Commit message: gripper added to cobot model

File: src/cobot_model/urdf/festo_cobot_model.urdf (robot description, URDF)
Before this commit: robot cobot_clean, 14 links, 13 joints
Links:
- removed link segment7_black
- removed link segment7_silver
- added link finger1, mass 0.001; collision mesh filename=package://cobot_model/meshes/v2_0_hull/finger01.stl scale=0.000001 0.000001 0.000001; visual mesh filename=package://cobot_model/meshes/v2_0_hull/finger01.stl scale=0.000001 0.000001 0.000001
- added link finger2, mass 0.001; collision mesh filename=package://cobot_model/meshes/v2_0_hull/finger02.stl scale=0.000001 0.000001 0.000001; visual mesh filename=package://cobot_model/meshes/v2_0_hull/finger02.stl scale=0.000001 0.000001 0.000001
- link segment7: mass None -> 0.1; geometry collision mesh filename=package://cobot_model/meshes/v2_0_hull/segment07_black.stl scale=0.001 0.001 0.001; visual mesh filename=package://cobot_model/meshes/v2_0_hull/segment07_black.stl scale=0.001 0.001 0.001
Joints:
- removed joint JFix_seg7_black
- removed joint JFix_seg7_silver
- added joint finger1_joint: type prismatic, parent TCP, child finger1, origin xyz=0.000000 0.0000 0.000000 rpy=0.0 0.0 0.0, axis 0 1 0, limit lower=-0.01 upper=0.015 effort=30.0 velocity=0.1
- added joint finger2_joint: type prismatic, parent TCP, child finger2, origin xyz=0.000000 0.0000 0.000000 rpy=0.0 0.0 0.0, axis 0 1 0, limit lower=-0.01 upper=0.015 effort=30.0 velocity=0.1
