Commit message: change controller of gripper from traj to command

File: src/cobot_model/urdf/gz_ros_controls.urdf.xacro (robot description, xacro)
@@ -161,5 +161,6 @@
     </joint>
     <joint name="finger2_joint">
-      <command_interface name="position"/>
+      <param name="mimic">finger1_joint</param>
+      <param name="multiplier">1</param>
       <state_interface name="position"/>
       <state_interface name="velocity"/>

File: src/cobot_model/urdf/robot_model.urdf.xacro (robot description, xacro)
@@ -344,5 +344,5 @@
         <parent link="TCP" />
         <child link="finger1" />
-        <axis xyz="0 1 0" />
+        <axis xyz="0 -1 0" />
         <limit effort="30.0" velocity="0.1" lower="-0.01" upper="0.015" />
     </joint>
@@ -353,4 +353,5 @@
         <axis xyz="0 1 0" />
         <limit effort="30.0" velocity="0.1" lower="-0.01" upper="0.015" />
+        <mimic joint="finger1_joint" />
     </joint>
 </robot>

Commit message: add vacuum gripper controllers

File: src/cobot_model/urdf/gz_ros_controls.urdf.xacro (robot description, xacro)
@@ -167,4 +167,17 @@
       <state_interface name="effort"/>
     </joint>
+     <joint name="vacuum_up_joint">
+      <command_interface name="position"/>
+      <state_interface name="position"/>
+      <state_interface name="velocity"/>
+      <state_interface name="effort"/>
+    </joint>
+    <joint name="vacuum_down_joint">
+      <param name="mimic">vacuum_up_joint</param>
+      <param name="multiplier">1</param>
+      <state_interface name="position"/>
+      <state_interface name="velocity"/>
+      <state_interface name="effort"/>
+    </joint>
   </ros2_control>
     <xacro:if value="${'gz' in '$(arg ros2_controls_plugin)'}">

Commit message: create controller for each vacuum gripper joint

File: src/cobot_model/urdf/gz_ros_controls.urdf.xacro (robot description, xacro)
@@ -157,6 +157,5 @@
     </joint>
     <joint name="vacuum_down_joint">
-      <param name="mimic">vacuum_up_joint</param>
-      <param name="multiplier">1</param>
+      <command_interface name="position"/>
       <state_interface name="position"/>
       <state_interface name="velocity"/>

File: src/cobot_model/urdf/robot_model.urdf.xacro (robot description, xacro)
@@ -501,5 +501,4 @@
         <axis xyz="0 1 1"/>
         <limit effort="30.0" lower="-0.01" upper="0.036" velocity="0.1"/>
-        <mimic joint="vacuum_up_joint"/>
     </joint>
 </robot>
