Commit message: add realsense to URDF

File: src/cobot_model/urdf/festo_cobot_model.urdf.xacro (robot description, xacro)
@@ -3,3 +3,13 @@
   <xacro:include filename="$(find cobot_model)/urdf/robot_model.urdf.xacro"/>
   <xacro:include filename="$(find cobot_model)/urdf/gz_ros_controls.urdf.xacro"/>
+  <xacro:arg name="enable_realsense_camera" default="false" />
+  <xacro:if value="${'$(arg enable_realsense_camera)' == 'true'}">
+    <xacro:arg name="use_nominal_extrinsics" default="true"/>
+    <xacro:arg name="add_plug" default="true" />
+    <xacro:arg name="use_mesh" default="true" />
+    <xacro:include filename="$(find realsense2_description)/urdf/_d435.urdf.xacro" />
+    <xacro:sensor_d435 parent="base_link" use_nominal_extrinsics="$(arg use_nominal_extrinsics)" add_plug="$(arg add_plug)" use_mesh="$(arg use_mesh)">
+      <origin xyz="-0.4 0.0 1.2" rpy="0.0 0.0 1.57"/>
+    </xacro:sensor_d435>
+  </xacro:if>
 </robot>

Commit message: added cobot model esslingen

File: src/cobot_model/urdf/festo_cobot_model.urdf.xacro (robot description, xacro)
@@ -1,4 +1,4 @@
 <?xml version="1.0" ?>
-<robot xmlns:xacro="http://www.ros.org/wiki/xacro" name="cobot_champion">
+<robot xmlns:xacro="http://www.ros.org/wiki/xacro" name="cobot_esslingen">
   <xacro:include filename="$(find cobot_model)/urdf/robot_model.urdf.xacro"/>
   <xacro:include filename="$(find cobot_model)/urdf/gz_ros_controls.urdf.xacro"/>

File: src/cobot_model/urdf/robot_model.urdf.xacro (robot description, xacro)
@@ -58,5 +58,5 @@
              <origin rpy="0.0 0.0 0.0" xyz="0.0 0.0 0.0" />
             <geometry>
-                <mesh filename="package://cobot_model/meshes/visual/segment01_visual.stl" scale="0.001 0.001 0.001" />
+                <mesh filename="package://cobot_model/meshes/visual/segment_01_logo.dae" scale="0.001 0.001 0.001" />
             </geometry>
             <material name="segment1_material">
@@ -83,5 +83,5 @@
             </geometry>
             <material name="segment2_material">
-                <color rgba="1.0 1.0 1.0 1.0" />
+                <color rgba="0 0.6 1.0 1.0" />
             </material>
         </visual>
@@ -105,5 +105,5 @@
             </geometry>
             <material name="segment3_material">
-                <color rgba="0.89 0.133 0.098 1.0" />
+               <color rgba="0.835 0.059 0.235 1.0" />
             </material>
         </visual>
@@ -127,5 +127,5 @@
             </geometry>
             <material name="segment4_material">
-                <color rgba="0.89 0.133 0.098 1.0" />
+                <color rgba="0.004 0.176 0.353 1.0" />
             </material>
         </visual>
@@ -149,5 +149,5 @@
             </geometry>
             <material name="segment5_material">
-                <color rgba="1.0 0.929 0.0 1.0" />
+                <color rgba="0 0.6 1.0 1.0" />
             </material>
         </visual>
@@ -171,5 +171,5 @@
             </geometry>
             <material name="segment6_material">
-                <color rgba="1.0 1.0 1.0 1.0" />
+                <color rgba="0.835 0.059 0.235 1.0" />
             </material>
         </visual>
@@ -275,5 +275,5 @@
         <child link="lin_axis_carriage" />
         <axis xyz="0 0 1" />
-        <limit effort="300.0" velocity="3.141593" lower="-.35" upper=".55" />
+        <limit effort="300.0" velocity="3.141593" lower="-.29" upper=".55" />
     </joint>
     <joint name="mount_fixture" type="fixed">
@@ -295,5 +295,5 @@
         <child link="segment3" />
         <axis xyz="0 0 1" />
-        <limit effort="150.0" velocity="3.141593" lower="-0.9" upper="1.570796" />
+        <limit effort="150.0" velocity="3.141593" lower="-0.9" upper="2.35" />
         <dynamics damping="0.0" friction="0.0" />
     </joint>
@@ -303,5 +303,5 @@
         <child link="segment4" />
         <axis xyz="0 0 1" />
-        <limit effort="100.0" velocity="3.141593" lower="-1.570796" upper="1.570796" />
+        <limit effort="100.0" velocity="3.141593" lower="-2.35" upper="1.570796" />
         <dynamics damping="0.0" friction="0.0" />
     </joint>
@@ -327,5 +327,5 @@
         <child link="segment7"/>
         <axis xyz="0 0 1"/>
-        <limit effort="20." lower="-2.356194" upper="2.356194" velocity="3.141593"/>
+        <limit effort="20." lower="-3.1" upper="3.1" velocity="3.141593"/>
         <dynamics damping="0.0" friction="0.0"/>
     </joint>

Commit message: updated calibrated camera params, V0

File: src/cobot_model/urdf/festo_cobot_model.urdf.xacro (robot description, xacro)
@@ -10,5 +10,5 @@
     <xacro:include filename="$(find realsense2_description)/urdf/_d435.urdf.xacro" />
     <xacro:sensor_d435 parent="base_link" use_nominal_extrinsics="$(arg use_nominal_extrinsics)" add_plug="$(arg add_plug)" use_mesh="$(arg use_mesh)">
-      <origin xyz="-0.4 0.0 1.2" rpy="0.0 0.0 1.57"/>
+      <origin xyz="-0.659 -0.459 1.550" rpy="2.999 0.787 1.371"/>
     </xacro:sensor_d435>
   </xacro:if>

Commit message: rotate camera frame

File: src/cobot_model/urdf/festo_cobot_model.urdf.xacro (robot description, xacro)
@@ -10,5 +10,5 @@
     <xacro:include filename="$(find realsense2_description)/urdf/_d435.urdf.xacro" />
     <xacro:sensor_d435 parent="base_link" use_nominal_extrinsics="$(arg use_nominal_extrinsics)" add_plug="$(arg add_plug)" use_mesh="$(arg use_mesh)">
-      <origin xyz="-0.659 -0.459 1.550" rpy="2.999 0.787 1.371"/>
+      <origin xyz="0.659 0.459 1.550" rpy="2.999 0.787 -1.771"/>
     </xacro:sensor_d435>
   </xacro:if>

Commit message: working calib params

File: src/cobot_model/urdf/festo_cobot_model.urdf.xacro (robot description, xacro)
@@ -5,10 +5,10 @@
   <xacro:arg name="enable_realsense_camera" default="false" />
   <xacro:if value="${'$(arg enable_realsense_camera)' == 'true'}">
-    <xacro:arg name="use_nominal_extrinsics" default="true"/>
+    <xacro:arg name="use_nominal_extrinsics" default="false"/>
     <xacro:arg name="add_plug" default="true" />
     <xacro:arg name="use_mesh" default="true" />
     <xacro:include filename="$(find realsense2_description)/urdf/_d435.urdf.xacro" />
-    <xacro:sensor_d435 parent="base_link" use_nominal_extrinsics="$(arg use_nominal_extrinsics)" add_plug="$(arg add_plug)" use_mesh="$(arg use_mesh)">
-      <origin xyz="0.659 0.459 1.550" rpy="2.999 0.787 -1.771"/>
+    <xacro:sensor_d435 parent="world" use_nominal_extrinsics="$(arg use_nominal_extrinsics)" add_plug="$(arg add_plug)" use_mesh="$(arg use_mesh)">
+      <origin xyz="0.441 0.319 1.378" rpy="-0.155 0.843 -1.727"/>
     </xacro:sensor_d435>
   </xacro:if>
