Commit message: use xacro for urdf creation

File: src/cobot_model/urdf/robot_model.urdf.xacro (robot description, xacro)
@@ -1,4 +1,4 @@
 <?xml version="1.0" ?>
-<robot name="cobot_zebra">
+<robot xmlns:xacro="http://www.ros.org/wiki/xacro">
     <link name="world" />
     <joint name="robot_in_world" type="fixed">
@@ -262,10 +262,10 @@
             </material>
         </visual>
-        <collision>
+       <!-- <collision>
             <origin xyz="-0.005 -0.002 0.010" rpy = "0 0 0" />
             <geometry>
                 <cylinder radius="0.00001" length="0.000001" />
             </geometry>
-        </collision>
+        </collision> -->
     </link>
     <!-- Joints -->

Commit message: handle all transformations in robot model within joints

File: src/cobot_model/urdf/robot_model.urdf.xacro (robot description, xacro)
@@ -3,5 +3,5 @@
     <link name="world" />
     <joint name="robot_in_world" type="fixed">
-        <origin xyz="0.0 0.0 0.3" rpy="0.0 0.0 0.0" />
+        <origin xyz="0.0 0.0 0.0" rpy="0.0 0.0 0.0" />
         <parent link="world" />
         <child link="base_link" />
@@ -12,5 +12,5 @@
     <link name="lin_axis">
         <visual>
-            <origin rpy="-1.570796327 3.141592654 0.0" xyz="0.0 -0.5 -0.32" />
+            <origin rpy="0.0 0.0 0.0" xyz="0.0 0.0 0.0" />
             <geometry>
                 <mesh filename="package://cobot_model/meshes/lin_axis/axis.dae" scale="0.001 0.001 0.001" />
@@ -21,5 +21,5 @@
         </visual>
         <collision>
-            <origin rpy="-1.570796327 3.141592654 0.0" xyz="0.0 -0.5 -0.32" />
+            <origin rpy="0.0 0.0 0.0" xyz="0.0 0.0 0.0" />
             <geometry>
                 <mesh filename="package://cobot_model/meshes/lin_axis/axis.dae" scale="0.001 0.001 0.001" />
@@ -28,5 +28,5 @@
         <inertial>
             <mass value="100.1" />
-            <origin rpy="-1.570796327 3.141592654 0.0" xyz="0.0 -0.5 -0.32" />
+            <origin rpy="0.0 0.0 0.0" xyz="0.0 0.0 0.0" />
             <inertia ixx="0.3" iyy="0.3" izz="0.3" ixy="0.0" ixz="0.0" iyz="0.0" />
         </inertial>
@@ -34,5 +34,5 @@
     <link name="lin_axis_carriage">
         <visual>
-            <origin rpy="-1.570796327 3.141592654 0.0" xyz="0.0 0.0 -0.32" />
+             <origin rpy="0.0 0.0 0.0" xyz="0.0 0.0 0.0" />
             <geometry>
                 <mesh filename="package://cobot_model/meshes/lin_axis/carriage.dae" scale="0.001 0.001 0.001" />
@@ -43,5 +43,5 @@
         </visual>
         <collision>
-            <origin rpy="-1.570796327 3.141592654 0.0" xyz="0.0 0.0 -0.32" />
+             <origin rpy="0.0 0.0 0.0" xyz="0.0 0.0 0.0" />
             <geometry>
                 <mesh filename="package://cobot_model/meshes/lin_axis/carriage.dae" scale="0.001 0.001 0.001" />
@@ -50,5 +50,5 @@
         <inertial>
             <mass value="1.0" />
-            <origin rpy="-1.570796327 3.141592654 0.0" xyz="0.0 0.0 -0.32" />
+             <origin rpy="0.0 0.0 0.0" xyz="0.0 0.0 0.0" />
             <inertia ixx="0.003" iyy="0.003" izz="0.003" ixy="0.0" ixz="0.0" iyz="0.0" />
         </inertial>
@@ -56,5 +56,5 @@
     <link name="segment1">
         <visual>
-            <origin rpy="-1.570793 -0.0 3.141593" xyz="0.0 -0.311 0.0" />
+             <origin rpy="0.0 0.0 0.0" xyz="0.0 0.0 0.0" />
             <geometry>
                 <mesh filename="package://cobot_model/meshes/v2_0_hull/segment01_combined.stl" scale="0.001 0.001 0.001" />
@@ -65,5 +65,5 @@
         </visual>
         <collision>
-            <origin rpy="-1.570793 0.0 3.141593" xyz="0.0 -0.311 0.0" />
+            <origin rpy="0.0 0.0 0.0" xyz="0.0 0.0 0.0" />
             <geometry>
                 <mesh filename="package://cobot_model/meshes/v2_0_hull/segment01_combined.stl" scale="0.001 0.001 0.001" />
@@ -72,5 +72,5 @@
         <inertial>
             <mass value="2.0" />
-            <origin rpy="-1.570793 0.0 3.141593" xyz="0.0 -0.311 0.0" />
+             <origin rpy="0.0 0.0 0.0" xyz="0.0 0.0 0.0" />
             <inertia ixx="0.0075496764161139766" iyy="0.009" izz="0.007" ixy="0.0" ixz="0.0" iyz="0.0" />
         </inertial>
@@ -78,5 +78,5 @@
     <link name="segment2">
         <visual>
-            <origin rpy="0.0 0.0 3.1415" xyz="0.0 0.0 0.036" />
+            <origin rpy="0.0 0.0 0.0" xyz="0.0 0.0 0.0" />
             <geometry>
                 <mesh filename="package://cobot_model/meshes/v2_0_hull/segment02_combined.stl" scale="0.001 0.001 0.001" />
@@ -87,5 +87,5 @@
         </visual>
         <collision>
-            <origin rpy="0.0 0.0 3.1415" xyz="0.0 0.0 0.036" />
+            <origin rpy="0.0 0.0 0.0" xyz="0.0 0.0 0.0" />
             <geometry>
                 <mesh filename="package://cobot_model/meshes/v2_0_hull/segment02_combined.stl" scale="0.001 0.001 0.001" />
@@ -94,5 +94,5 @@
         <inertial>
             <mass value="1.0" />
-            <origin rpy="0.0 0.0 3.1415" xyz="0.0 0.0 0.036" />
+             <origin rpy="0.0 0.0 0.0" xyz="0.0 0.0 0.0" />
             <inertia ixx="0.03" iyy="0.03" izz="0.03" ixy="0.0" ixz="0.0" iyz="0.0" />
         </inertial>
@@ -100,5 +100,5 @@
     <link name="segment3">
         <visual>
-            <origin rpy="0.0 0.0 3.1415" xyz="0.001 0.0 0.06" />
+            <origin rpy="0.0 0.0 0.0" xyz="0.0 0.0 0.0" />
             <geometry>
                 <mesh filename="package://cobot_model/meshes/v2_0_hull/segment03_combined.stl" scale="0.001 0.001 0.001" />
@@ -109,5 +109,5 @@
         </visual>
         <collision>
-            <origin rpy="0.0 0.0 3.1415" xyz="0.001 0.0 0.06" />
+            <origin rpy="0.0 0.0 0.0" xyz="0.0 0.0 0.0" />
             <geometry>
                 <mesh filename="package://cobot_model/meshes/v2_0_hull/segment03_combined.stl" scale="0.001 0.001 0.001" />
@@ -116,5 +116,5 @@
         <inertial>
             <mass value="0.1" />
-            <origin rpy="0.0 0.0 3.1415" xyz="0.001 0.0 0.06" />
+            <origin rpy="0.0 0.0 0.0" xyz="0.0 0.0 0.0" />
             <inertia ixx="0.03" iyy="0.03" izz="0.03" ixy="0.0" ixz="0.0" iyz="0.0" />
         </inertial>
@@ -122,5 +122,5 @@
     <link name="segment4">
         <visual>
-            <origin rpy="3.1415 0.0 -1.5707 " xyz="0.0 0.0 -0.035" />
+            <origin rpy="0.0 0.0 0.0" xyz="0.0 0.0 0.0" />
             <geometry>
                 <mesh filename="package://cobot_model/meshes/v2_0_hull/segment04_combined.stl" scale="0.001 0.001 0.001" />
@@ -131,5 +131,5 @@
         </visual>
         <collision>
-            <origin rpy="3.1415 0.0 -1.5707 " xyz="0.0 0.0 -0.035" />
+             <origin rpy="0.0 0.0 0.0" xyz="0.0 0.0 0.0" />
             <geometry>
                 <mesh filename="package://cobot_model/meshes/v2_0_hull/segment04_combined.stl" scale="0.001 0.001 0.001" />
@@ -138,5 +138,5 @@
         <inertial>
             <mass value="1.0" />
-            <origin rpy="3.1415 0.0 -1.5707 " xyz="0.0 0.0 -0.035" />
+             <origin rpy="0.0 0.0 0.0" xyz="0.0 0.0 0.0" />
             <inertia ixx="0.003" iyy="0.003" izz="0.003" ixy="0.0" ixz="0.0" iyz="0.0" />
         </inertial>
@@ -144,5 +144,5 @@
     <link name="segment5">
         <visual>
-            <origin rpy="0.0 0.0 3.1415" xyz="0.0 0.0 0.015" />
+            <origin rpy="0.0 0.0 0.0" xyz="0.0 0.0 0.0" />
             <geometry>
                 <mesh filename="package://cobot_model/meshes/v2_0_hull/segment05_combined.stl" scale="0.001 0.001 0.001" />
@@ -153,5 +153,5 @@
         </visual>
         <collision>
-            <origin rpy="0.0 0.0 3.1415" xyz="0.0 0.0 0.015" />
+            <origin rpy="0.0 0.0 0.0" xyz="0.0 0.0 0.0" />
             <geometry>
                 <mesh filename="package://cobot_model/meshes/v2_0_hull/segment05_combined.stl" scale="0.001 0.001 0.001" />
@@ -160,5 +160,5 @@
         <inertial>
             <mass value="0.5" />
-            <origin rpy="0.0 0.0 3.1415" xyz="0.0 0.0 0.015" />
+            <origin rpy="0.0 0.0 0.0" xyz="0.0 0.0 0.0" />
             <inertia ixx="0.001" iyy="0.001" izz="0.001" ixy="0.0" ixz="0.0" iyz="0.0" />
         </inertial>
@@ -166,5 +166,5 @@
     <link name="segment6">
         <visual>
-            <origin rpy="0.0 0.0 -1.5708" xyz="0.005 0.0 0.038" />
+            <origin rpy="0.0 0.0 0.0" xyz="0.0 0.0 0.0" />
             <geometry>
                 <mesh filename="package://cobot_model/meshes/v2_0_hull/segment06_combined.stl" scale="0.001 0.001 0.001" />
@@ -175,5 +175,5 @@
         </visual>
         <collision>
-            <origin rpy="0.0 0.0 -1.5708" xyz="0.005 0.0 0.038" />
+            <origin rpy="0.0 0.0 0.0" xyz="0.0 0.0 0.0" />
             <geometry>
                 <mesh filename="package://cobot_model/meshes/v2_0_hull/segment06_combined.stl" scale="0.001 0.001 0.001" />
@@ -182,5 +182,5 @@
         <inertial>
             <mass value="0.1" />
-            <origin rpy="0.0 0.0 -1.5708" xyz="0.005 0.0 0.038" />
+            <origin rpy="0.0 0.0 0.0" xyz="0.0 0.0 0.0" />
             <inertia ixx="0.03" iyy="0.03" izz="0.03" ixy="0.0" ixz="0.0" iyz="0.0" />
         </inertial>
@@ -188,5 +188,5 @@
     <link name="segment7">
         <visual>
-            <origin rpy="0.0 0.0 0.0" xyz="0.004 0.002 0.091" />
+            <origin rpy="0.0 0.0 0.0" xyz="0.0 0.0 0.0" />
             <material name="Aterul">
                 <color rgba="0.0 0.0 0.0 1.0" />
@@ -197,5 +197,5 @@
         </visual>
         <collision>
-            <origin rpy="0.0 0.0 0.0" xyz="0.004 0.002 0.091" />
+            <origin rpy="0.0 0.0 0.0" xyz="0.0 0.0 0.0" />
             <geometry>
                 <mesh filename="package://cobot_model/meshes/v2_0_hull/segment07_black.stl" scale="0.001 0.001 0.001" />
@@ -204,14 +204,31 @@
         <inertial>
             <mass value="0.1" />
-            <origin rpy="0.0 0.0 0.0" xyz="0.004 0.002 0.091" />
+            <origin rpy="0.0 0.0 0.0" xyz="0.0 0.0 0.0" />
             <inertia ixx="0.03" iyy="0.03" izz="0.03" ixy="0.0" ixz="0.0" iyz="0.0" />
         </inertial>
     </link>
-    <link name="finger1">
-        <visual>
-            <origin rpy="0.0 -0.000000 0.000000" xyz="0.0 0.0 0.0" />
+    <link name="TCP">
+        <visual>
+            <origin rpy="0.0 0.0 0.0" xyz="0.0 0.0 0.0" />
+            <geometry>
+                <cylinder radius="0.00001" length="0.000001" />
+            </geometry>
             <material name="silver">
                 <color rgba="0.629 0.629 0.625 1.0" />
             </material>
+        </visual>
+        <collision>
+            <origin rpy="0.0 0.0 0.0" xyz="0.0 0.0 0.0" />
+            <geometry>
+                <cylinder radius="0.0001" length="0.0001" />
+            </geometry>
+        </collision>
+    </link>
+    <link name="finger1">
+        <visual>
+            <origin rpy="0.0 0.0 0.0" xyz="0.0 0.0 0.0" />
+            <material name="silver">
+                <color rgba="0.629 0.629 0.625 1.0" />
+            </material>
             <geometry>
                 <mesh filename="package://cobot_model/meshes/v2_0_hull/finger01.stl" scale="0.000001 0.000001 0.000001" />
@@ -219,5 +236,5 @@
         </visual>
         <collision>
-            <origin rpy="0.0 -0.000000 0.000000" xyz="0.0 0.0 0.0" />
+            <origin rpy="0.0 0.0 0.0" xyz="0.0 0.0 0.0" />
             <geometry>
                 <mesh filename="package://cobot_model/meshes/v2_0_hull/finger01.stl" scale="0.000001 0.000001 0.000001" />
@@ -232,5 +249,5 @@
     <link name="finger2">
         <visual>
-            <origin rpy="0.0 -0.000000 0.000000" xyz="0.0 0.0 0.0" />
+            <origin rpy="0.0 0.0 0.0" xyz="0.0 0.0 0.0" />
             <material name="silver">
                 <color rgba="0.629 0.629 0.625 1.0" />
@@ -241,5 +258,5 @@
         </visual>
         <collision>
-            <origin rpy="0.0 -0.000000 0.000000" xyz="0.0 0.0 0.0" />
+            <origin rpy="0.0 0.0 0.0" xyz="0.0 0.0 0.0" />
             <geometry>
                 <mesh filename="package://cobot_model/meshes/v2_0_hull/finger02.stl" scale="0.000001 0.000001 0.000001" />
@@ -252,36 +269,19 @@
         </inertial>
     </link>
-    <link name="TCP">
-        <visual>
-            <origin xyz="-0.005 -0.002 0.01" rpy="0.0 0.0 0.0" />
-            <geometry>
-                <cylinder radius="0.00001" length="0.000001" />
-            </geometry>
-            <material name="silver">
-                <color rgba="0.629 0.629 0.625 1.0" />
-            </material>
-        </visual>
-       <!-- <collision>
-            <origin xyz="-0.005 -0.002 0.010" rpy = "0 0 0" />
-            <geometry>
-                <cylinder radius="0.00001" length="0.000001" />
-            </geometry>
-        </collision> -->
-    </link>
     <!-- Joints -->
     <joint name="joint_0" type="prismatic">
-        <origin rpy="0.0 0.0 0.0" xyz="0.0 0.0 0.0" />
+        <origin rpy="0.0 0.0 0.0" xyz="0.0 0.0 0.3" />
         <parent link="lin_axis" />
         <child link="lin_axis_carriage" />
-        <axis xyz="0 1 0" />
+        <axis xyz="0 0 1" />
         <limit effort="200.000" velocity="3.141593" lower="-.35" upper=".55" />
     </joint>
     <joint name="mount_fixture" type="fixed">
-        <origin rpy="0.0 0.0 0.0" xyz="0.0 0.0 0.0" />
+        <origin rpy="0.0 0.0 0.0" xyz="0.0 0.3 0.3" />
         <parent link="lin_axis_carriage" />
         <child link="segment1" />
     </joint>
     <joint name="joint_1" type="revolute">
-        <origin rpy="-1.570793 0.0 3.141593" xyz="0.0 -0.274400 0.0" />
+        <origin rpy="0.0 0.0 0.0" xyz="0.0 0.0 0.0" />
         <parent link="segment1" />
         <child link="segment2" />
@@ -291,5 +291,5 @@
     </joint>
     <joint name="joint_2" type="revolute">
-        <origin rpy="-1.570796 0.0 0.0" xyz="0.00005 0.04955 0.1555" />
+        <origin rpy="1.5708 0.0 0.0" xyz="0.0 -0.111 0.118" />
         <parent link="segment2" />
         <child link="segment3" />
@@ -299,5 +299,5 @@
     </joint>
     <joint name="joint_3" type="revolute">
-        <origin rpy="3.141593 0.0 1.570796" xyz="-0.254493 0.0 0.0852" />
+        <origin rpy="0.0 0.0 0.0" xyz="0.254 0.0 0.06" />
         <parent link="segment3" />
         <child link="segment4" />
@@ -307,5 +307,5 @@
     </joint>
     <joint name="joint_4" type="revolute">
-        <origin rpy="-1.570796 0.0 -3.141593" xyz="0.0 -0.0076 0.132393" />
+        <origin rpy="-1.5708 0.0 -1.5708" xyz="0.024 0.0 -0.168" />
         <parent link="segment4" />
         <child link="segment5" />
@@ -315,5 +315,5 @@
     </joint>
     <joint name="joint_5" type="revolute">
-        <origin rpy="-1.570796 0.0 3.141593" xyz="0.0 -0.0063 0.113264" />
+        <origin rpy="-1.570 -1.570 0.0" xyz="0.0 0.042 0.103" />
         <parent link="segment5" />
         <child link="segment6" />
@@ -323,5 +323,5 @@
     </joint>
     <joint name="joint_6" type="revolute">
-        <origin rpy="1.570796 0.0 0.0" xyz="0.0 -0.1328 -0.006164" />
+        <origin rpy="0.0 -1.570 0.0" xyz="0.26 0.0 -0.041" />
         <parent link="segment6" />
         <child link="segment7" />
@@ -331,15 +331,15 @@
     </joint>
     <joint name="JFix_TCP" type="fixed">
-        <origin rpy="0.0 0.0 3.141593" xyz="0.0 0.0 0.190143" />
+        <origin rpy="0.0 3.141593 0.0" xyz="0.0 0.0 -0.06" />
         <parent link="segment7" />
         <child link="TCP" />
     </joint>
-    <joint name="JFix_Base" type="fixed">
-        <origin rpy="-1.570796 0.0 0.0" xyz="0.0 0.0 0.5" />
+   <joint name="JFix_Base" type="fixed">
+        <origin rpy="0.0 0.0 0.0" xyz="0.0 0.0 0.0" />
         <parent link="base_link" />
         <child link="lin_axis" />
     </joint>
     <joint name="finger1_joint" type="prismatic">
-        <origin rpy="0.0 0.0 0.0" xyz="0.000000 0.0000 0.000000" />
+        <origin rpy="0.0 0.0 0.0" xyz="0.0 0.0 0.0" />
         <parent link="TCP" />
         <child link="finger1" />
@@ -348,5 +348,5 @@
     </joint>
     <joint name="finger2_joint" type="prismatic">
-        <origin rpy="0.0 0.0 0.0" xyz="0.000000 0.0000 0.000000" />
+        <origin rpy="0.0 0.0 0.0" xyz="0.0 0.0 0.0" />
         <parent link="TCP" />
         <child link="finger2" />
