Commit message: re-defined inertial values for cobot

File: src/cobot_model/urdf/robot_model.urdf.xacro (robot description, xacro)
@@ -27,7 +27,7 @@
         </collision>
         <inertial>
-            <mass value="100.1" />
-            <origin rpy="0.0 0.0 0.0" xyz="0.0 0.0 0.0" />
-            <inertia ixx="0.3" iyy="0.3" izz="0.3" ixy="0.0" ixz="0.0" iyz="0.0" />
+            <mass value="8.6" />
+            <origin rpy="0.0 0.0 0.0" xyz="0.0 0.0 0.6" />
+            <inertia ixx="1.03466672" iyy="1.0433778" izz="0.01404452" ixy="0.0" ixz="0.0" iyz="0.0" />
         </inertial>
     </link>
@@ -49,7 +49,7 @@
         </collision>
         <inertial>
-            <mass value="1.0" />
-             <origin rpy="0.0 0.0 0.0" xyz="0.0 0.0 0.0" />
-            <inertia ixx="0.003" iyy="0.003" izz="0.003" ixy="0.0" ixz="0.0" iyz="0.0" />
+            <mass value="0.7" />
+            <origin rpy="0.0 0.0 0.0" xyz="0.0 0.0 0.11" />
+            <inertia ixx="0.00287479" iyy="0.00415339" izz="0.00138151" ixy="0.0" ixz="0.0" iyz="0.0" />
         </inertial>
     </link>
@@ -71,7 +71,7 @@
         </collision>
         <inertial>
-            <mass value="2.0" />
-             <origin rpy="0.0 0.0 0.0" xyz="0.0 0.0 0.0" />
-            <inertia ixx="0.0075496764161139766" iyy="0.009" izz="0.007" ixy="0.0" ixz="0.0" iyz="0.0" />
+            <mass value="7.3" />
+             <origin rpy="0.0 0.0 0.0" xyz="0.0 0.0 -0.156" />
+            <inertia ixx="0.0697588" iyy="0.0697588" izz="0.0210824" ixy="0.0" ixz="0.0" iyz="0.0" />
         </inertial>
     </link>
@@ -93,7 +93,7 @@
         </collision>
         <inertial>
-            <mass value="1.0" />
-             <origin rpy="0.0 0.0 0.0" xyz="0.0 0.0 0.0" />
-            <inertia ixx="0.03" iyy="0.03" izz="0.03" ixy="0.0" ixz="0.0" iyz="0.0" />
+            <mass value="5.0" />
+            <origin rpy="0.0 0.0 0.0" xyz="0.0 0.0 0.119" />
+            <inertia ixx="0.03441292" iyy="0.02442542" izz="0.03361208" ixy="0.0" ixz="0.0" iyz="0.0" />
         </inertial>
     </link>
@@ -115,7 +115,7 @@
         </collision>
         <inertial>
-            <mass value="0.1" />
-            <origin rpy="0.0 0.0 0.0" xyz="0.0 0.0 0.0" />
-            <inertia ixx="0.03" iyy="0.03" izz="0.03" ixy="0.0" ixz="0.0" iyz="0.0" />
+            <mass value="1.0" />
+            <origin rpy="0.0 0.0 0.0" xyz="0.126 0.0 0.06" />
+            <inertia ixx="0.00530033" ixy="0.0" ixz="-0.00756" iyy="0.02606333" iyz="0.0" izz="0.02242967" />
         </inertial>
     </link>
@@ -137,7 +137,7 @@
         </collision>
         <inertial>
-            <mass value="1.0" />
-             <origin rpy="0.0 0.0 0.0" xyz="0.0 0.0 0.0" />
-            <inertia ixx="0.003" iyy="0.003" izz="0.003" ixy="0.0" ixz="0.0" iyz="0.0" />
+            <mass value="3.4" />
+            <origin rpy="0.0 0.0 0.0" xyz="0.0 0.0 -0.112" />
+            <inertia ixx="0.01850875" ixy="0.0" ixz="0.0" iyy="0.01850875" iyz="0.0" izz="0.00833" />
         </inertial>
     </link>
@@ -159,7 +159,7 @@
         </collision>
         <inertial>
-            <mass value="0.5" />
-            <origin rpy="0.0 0.0 0.0" xyz="0.0 0.0 0.0" />
-            <inertia ixx="0.001" iyy="0.001" izz="0.001" ixy="0.0" ixz="0.0" iyz="0.0" />
+            <mass value="1.1" />
+            <origin rpy="0.0 0.0 0.0" xyz="0.0 0.0 0.071" />
+            <inertia ixx="0.00326077" iyy="0.00326077" izz="0.00277255" ixy="0.0" ixz="0.0" iyz="0.0" />
         </inertial>
     </link>
@@ -181,7 +181,7 @@
         </collision>
         <inertial>
-            <mass value="0.1" />
-            <origin rpy="0.0 0.0 0.0" xyz="0.0 0.0 0.0" />
-            <inertia ixx="0.03" iyy="0.03" izz="0.03" ixy="0.0" ixz="0.0" iyz="0.0" />
+            <mass value="1.5" />
+            <origin rpy="0.0 0.0 0.0" xyz="0.071 0.0 0.0" />
+            <inertia ixx="0.00319363" iyy="0.01012625" izz="0.01115763" ixy="0.0" ixz="0.0" iyz="0.0" />
         </inertial>
     </link>
@@ -203,7 +203,7 @@
         </collision>
         <inertial>
-            <mass value="0.1" />
-            <origin rpy="0.0 0.0 0.0" xyz="0.0 0.0 0.0" />
-            <inertia ixx="0.03" iyy="0.03" izz="0.03" ixy="0.0" ixz="0.0" iyz="0.0" />
+            <mass value="0.2" />
+            <origin rpy="0.0 0.0 0.0" xyz="0.0 0.0 0.0" />
+            <inertia ixx="0.00040667" iyy="0.00030104" izz="0.00059971" ixy="0.0" ixz="0.0" iyz="0.0" />
         </inertial>
     </link>
@@ -242,7 +242,7 @@
         </collision>
         <inertial>
-            <mass value="0.001" />
-            <inertia ixx="100.0" iyy="100.0" izz="100.0" ixy="0.0" ixz="0.0" iyz="0.0" />
-            <origin xyz="0.0 0.0 0.0" rpy="0.0 0.0 0.0" />
+            <mass value="0.05" />
+            <origin rpy="0.0 0.0 0.0" xyz="0.0 0.0 0.0" />
+            <inertia ixx="3.46666667e-05" iyy="2.64166667e-05" izz="1.78833333e-05" ixy="0.0" ixz="0.0" iyz="0.0" />
         </inertial>
     </link>
@@ -264,7 +264,7 @@
         </collision>
         <inertial>
-            <mass value="0.001" />
-            <inertia ixx="100.0" iyy="100.0" izz="100.0" ixy="0.0" ixz="0.0" iyz="0.0" />
-            <origin xyz="0.0 0.0 0.0" rpy="0.0 0.0 0.0" />
+            <mass value="0.05" />
+            <origin rpy="0.0 0.0 0.0" xyz="0.0 0.0 0.0" />
+            <inertia ixx="3.46666667e-05" iyy="2.64166667e-05" izz="1.78833333e-05" ixy="0.0" ixz="0.0" iyz="0.0" />
         </inertial>
     </link>
@@ -275,5 +275,5 @@
         <child link="lin_axis_carriage" />
         <axis xyz="0 0 1" />
-        <limit effort="200.000" velocity="3.141593" lower="-.35" upper=".55" />
+        <limit effort="200.0" velocity="3.141593" lower="-.35" upper=".55" />
     </joint>
     <joint name="mount_fixture" type="fixed">
@@ -295,5 +295,5 @@
         <child link="segment3" />
         <axis xyz="0 0 1" />
-        <limit effort="20.0" velocity="3.141593" lower="-1.570796" upper="1.570796" />
+        <limit effort="40.0" velocity="3.141593" lower="-1.570796" upper="1.570796" />
         <dynamics damping="0.0" friction="0.0" />
     </joint>
@@ -303,5 +303,5 @@
         <child link="segment4" />
         <axis xyz="0 0 1" />
-        <limit effort="10.0" velocity="3.141593" lower="-1.570796" upper="1.570796" />
+        <limit effort="40.0" velocity="3.141593" lower="-1.570796" upper="1.570796" />
         <dynamics damping="0.0" friction="0.0" />
     </joint>
@@ -311,5 +311,5 @@
         <child link="segment5" />
         <axis xyz="0 0 1" />
-        <limit effort="10.0" velocity="3.141593" lower="-1.570796" upper="1.570796" />
+        <limit effort="40.0" velocity="3.141593" lower="-1.570796" upper="1.570796" />
         <dynamics damping="0.0" friction="0.0" />
     </joint>
@@ -319,5 +319,5 @@
         <child link="segment6" />
         <axis xyz="0 0 1" />
-        <limit effort="10.0" velocity="3.141593" lower="-1.570796" upper="1.570796" />
+        <limit effort="40.0" velocity="3.141593" lower="-1.570796" upper="1.570796" />
         <dynamics damping="0.0" friction="0.0" />
     </joint>
@@ -327,5 +327,5 @@
         <child link="segment7" />
         <axis xyz="0 0 1" />
-        <limit effort="10." velocity="3.141593" lower="-2.356194" upper="2.356194" />
+        <limit effort="40." velocity="3.141593" lower="-2.356194" upper="2.356194" />
         <dynamics damping="0.0" friction="0.0" />
     </joint>

Commit message: fix segment 3 / 4 links and adjust effort limits (educated guess)

File: src/cobot_model/urdf/robot_model.urdf.xacro (robot description, xacro)
@@ -115,7 +115,7 @@
         </collision>
         <inertial>
-            <mass value="1.0" />
+            <mass value="2.5" />
             <origin rpy="0.0 0.0 0.0" xyz="0.126 0.0 0.06" />
-            <inertia ixx="0.00530033" ixy="0.0" ixz="-0.00756" iyy="0.02606333" iyz="0.0" izz="0.02242967" />
+            <inertia ixx="0.01325083" ixy="0.0" ixz="-0.0189" iyy="0.06515833" iyz="0.0" izz="0.05607417" />
         </inertial>
     </link>
@@ -182,5 +182,5 @@
         <inertial>
             <mass value="1.5" />
-            <origin rpy="0.0 0.0 0.0" xyz="0.071 0.0 0.0" />
+            <origin rpy="0.0 0.0 0.0" xyz="0.12 0.0 0.0" />
             <inertia ixx="0.00319363" iyy="0.01012625" izz="0.01115763" ixy="0.0" ixz="0.0" iyz="0.0" />
         </inertial>
@@ -275,5 +275,5 @@
         <child link="lin_axis_carriage" />
         <axis xyz="0 0 1" />
-        <limit effort="200.0" velocity="3.141593" lower="-.35" upper=".55" />
+        <limit effort="300.0" velocity="3.141593" lower="-.35" upper=".55" />
     </joint>
     <joint name="mount_fixture" type="fixed">
@@ -287,5 +287,5 @@
         <child link="segment2" />
         <axis xyz="0 0 1" />
-        <limit effort="40.0" velocity="3.141593" lower="-0.7853976732051033" upper="3.9269903267948965" />
+        <limit effort="200.0" velocity="3.141593" lower="-0.7853976732051033" upper="3.9269903267948965" />
         <dynamics damping="0.0" friction="0.0" />
     </joint>
@@ -295,5 +295,5 @@
         <child link="segment3" />
         <axis xyz="0 0 1" />
-        <limit effort="40.0" velocity="3.141593" lower="-1.570796" upper="1.570796" />
+        <limit effort="150.0" velocity="3.141593" lower="-1.570796" upper="1.570796" />
         <dynamics damping="0.0" friction="0.0" />
     </joint>
@@ -303,5 +303,5 @@
         <child link="segment4" />
         <axis xyz="0 0 1" />
-        <limit effort="40.0" velocity="3.141593" lower="-1.570796" upper="1.570796" />
+        <limit effort="100.0" velocity="3.141593" lower="-1.570796" upper="1.570796" />
         <dynamics damping="0.0" friction="0.0" />
     </joint>
@@ -311,5 +311,5 @@
         <child link="segment5" />
         <axis xyz="0 0 1" />
-        <limit effort="40.0" velocity="3.141593" lower="-1.570796" upper="1.570796" />
+        <limit effort="50.0" velocity="3.141593" lower="-1.570796" upper="1.570796" />
         <dynamics damping="0.0" friction="0.0" />
     </joint>
@@ -319,5 +319,5 @@
         <child link="segment6" />
         <axis xyz="0 0 1" />
-        <limit effort="40.0" velocity="3.141593" lower="-1.570796" upper="1.570796" />
+        <limit effort="50.0" velocity="3.141593" lower="-1.570796" upper="1.570796" />
         <dynamics damping="0.0" friction="0.0" />
     </joint>
@@ -327,5 +327,5 @@
         <child link="segment7" />
         <axis xyz="0 0 1" />
-        <limit effort="40." velocity="3.141593" lower="-2.356194" upper="2.356194" />
+        <limit effort="20." velocity="3.141593" lower="-2.356194" upper="2.356194" />
         <dynamics damping="0.0" friction="0.0" />
     </joint>

Commit message: reduced meshes for collisions added

File: src/cobot_model/urdf/robot_model.urdf.xacro (robot description, xacro)
@@ -23,5 +23,5 @@
             <origin rpy="0.0 0.0 0.0" xyz="0.0 0.0 0.0" />
             <geometry>
-                <mesh filename="package://cobot_model/meshes/lin_axis/axis.dae" scale="0.001 0.001 0.001" />
+                <mesh filename="package://cobot_model/meshes/collision/axis_collision.dae" scale="0.001 0.001 0.001" />
             </geometry>
         </collision>
@@ -45,5 +45,5 @@
              <origin rpy="0.0 0.0 0.0" xyz="0.0 0.0 0.0" />
             <geometry>
-                <mesh filename="package://cobot_model/meshes/lin_axis/carriage.dae" scale="0.001 0.001 0.001" />
+                <mesh filename="package://cobot_model/meshes/collision/carriage_collision.dae" scale="0.001 0.001 0.001" />
             </geometry>
         </collision>
@@ -67,5 +67,5 @@
             <origin rpy="0.0 0.0 0.0" xyz="0.0 0.0 0.0" />
             <geometry>
-                <mesh filename="package://cobot_model/meshes/v2_0_hull/segment01_combined.stl" scale="0.001 0.001 0.001" />
+                <mesh filename="package://cobot_model/meshes/collision/segment01_collision.stl" scale="0.001 0.001 0.001" />
             </geometry>
         </collision>
@@ -89,5 +89,5 @@
             <origin rpy="0.0 0.0 0.0" xyz="0.0 0.0 0.0" />
             <geometry>
-                <mesh filename="package://cobot_model/meshes/v2_0_hull/segment02_combined.stl" scale="0.001 0.001 0.001" />
+                <mesh filename="package://cobot_model/meshes/collision/segment02_collision.stl" scale="0.001 0.001 0.001" />
             </geometry>
         </collision>
@@ -111,5 +111,5 @@
             <origin rpy="0.0 0.0 0.0" xyz="0.0 0.0 0.0" />
             <geometry>
-                <mesh filename="package://cobot_model/meshes/v2_0_hull/segment03_combined.stl" scale="0.001 0.001 0.001" />
+                <mesh filename="package://cobot_model/meshes/collision/segment03_collision.stl" scale="0.001 0.001 0.001" />
             </geometry>
         </collision>
@@ -133,5 +133,5 @@
              <origin rpy="0.0 0.0 0.0" xyz="0.0 0.0 0.0" />
             <geometry>
-                <mesh filename="package://cobot_model/meshes/v2_0_hull/segment04_combined.stl" scale="0.001 0.001 0.001" />
+                <mesh filename="package://cobot_model/meshes/collision/segment04_collision.stl" scale="0.001 0.001 0.001" />
             </geometry>
         </collision>
@@ -155,5 +155,5 @@
             <origin rpy="0.0 0.0 0.0" xyz="0.0 0.0 0.0" />
             <geometry>
-                <mesh filename="package://cobot_model/meshes/v2_0_hull/segment05_combined.stl" scale="0.001 0.001 0.001" />
+                <mesh filename="package://cobot_model/meshes/collision/segment05_collision.stl" scale="0.001 0.001 0.001" />
             </geometry>
         </collision>
@@ -177,5 +177,5 @@
             <origin rpy="0.0 0.0 0.0" xyz="0.0 0.0 0.0" />
             <geometry>
-                <mesh filename="package://cobot_model/meshes/v2_0_hull/segment06_combined.stl" scale="0.001 0.001 0.001" />
+                <mesh filename="package://cobot_model/meshes/collision/segment06_collision.stl" scale="0.001 0.001 0.001" />
             </geometry>
         </collision>
@@ -199,5 +199,5 @@
             <origin rpy="0.0 0.0 0.0" xyz="0.0 0.0 0.0" />
             <geometry>
-                <mesh filename="package://cobot_model/meshes/v2_0_hull/segment07_black.stl" scale="0.001 0.001 0.001" />
+                <mesh filename="package://cobot_model/meshes/collision/segment07_collision.stl" scale="0.001 0.001 0.001" />
             </geometry>
         </collision>
@@ -238,5 +238,5 @@
             <origin rpy="0.0 0.0 0.0" xyz="0.0 0.0 0.0" />
             <geometry>
-                <mesh filename="package://cobot_model/meshes/v2_0_hull/finger01.stl" scale="0.000001 0.000001 0.000001" />
+                <mesh filename="package://cobot_model/meshes/collision/finger01_collision.stl" scale="0.000001 0.000001 0.000001" />
             </geometry>
         </collision>
@@ -260,5 +260,5 @@
             <origin rpy="0.0 0.0 0.0" xyz="0.0 0.0 0.0" />
             <geometry>
-                <mesh filename="package://cobot_model/meshes/v2_0_hull/finger02.stl" scale="0.000001 0.000001 0.000001" />
+                <mesh filename="package://cobot_model/meshes/collision/finger02_collision.stl" scale="0.000001 0.000001 0.000001" />
             </geometry>
         </collision>

Commit message: cleanup visual meshes

File: src/cobot_model/urdf/robot_model.urdf.xacro (robot description, xacro)
@@ -14,5 +14,5 @@
             <origin rpy="0.0 0.0 0.0" xyz="0.0 0.0 0.0" />
             <geometry>
-                <mesh filename="package://cobot_model/meshes/lin_axis/axis.dae" scale="0.001 0.001 0.001" />
+                <mesh filename="package://cobot_model/meshes/visual/axis_visual.dae" scale="0.001 0.001 0.001" />
                 <material name="silver">
                     <color rgba="1.0 1.0 1.0 1.0" />
@@ -36,5 +36,5 @@
              <origin rpy="0.0 0.0 0.0" xyz="0.0 0.0 0.0" />
             <geometry>
-                <mesh filename="package://cobot_model/meshes/lin_axis/carriage.dae" scale="0.001 0.001 0.001" />
+                <mesh filename="package://cobot_model/meshes/visual/carriage_visual.dae" scale="0.001 0.001 0.001" />
                 <material name="silver">
                     <color rgba="1.0 1.0 1.0 1.0" />
@@ -58,5 +58,5 @@
              <origin rpy="0.0 0.0 0.0" xyz="0.0 0.0 0.0" />
             <geometry>
-                <mesh filename="package://cobot_model/meshes/v2_0_hull/segment01_combined.stl" scale="0.001 0.001 0.001" />
+                <mesh filename="package://cobot_model/meshes/visual/segment01_visual.stl" scale="0.001 0.001 0.001" />
             </geometry>
             <material name="segment1_material">
@@ -80,5 +80,5 @@
             <origin rpy="0.0 0.0 0.0" xyz="0.0 0.0 0.0" />
             <geometry>
-                <mesh filename="package://cobot_model/meshes/v2_0_hull/segment02_combined.stl" scale="0.001 0.001 0.001" />
+                <mesh filename="package://cobot_model/meshes/visual/segment02_visual.stl" scale="0.001 0.001 0.001" />
             </geometry>
             <material name="segment2_material">
@@ -102,5 +102,5 @@
             <origin rpy="0.0 0.0 0.0" xyz="0.0 0.0 0.0" />
             <geometry>
-                <mesh filename="package://cobot_model/meshes/v2_0_hull/segment03_combined.stl" scale="0.001 0.001 0.001" />
+                <mesh filename="package://cobot_model/meshes/visual/segment03_visual.stl" scale="0.001 0.001 0.001" />
             </geometry>
             <material name="segment3_material">
@@ -124,5 +124,5 @@
             <origin rpy="0.0 0.0 0.0" xyz="0.0 0.0 0.0" />
             <geometry>
-                <mesh filename="package://cobot_model/meshes/v2_0_hull/segment04_combined.stl" scale="0.001 0.001 0.001" />
+                <mesh filename="package://cobot_model/meshes/visual/segment04_visual.stl" scale="0.001 0.001 0.001" />
             </geometry>
             <material name="segment4_material">
@@ -146,5 +146,5 @@
             <origin rpy="0.0 0.0 0.0" xyz="0.0 0.0 0.0" />
             <geometry>
-                <mesh filename="package://cobot_model/meshes/v2_0_hull/segment05_combined.stl" scale="0.001 0.001 0.001" />
+                <mesh filename="package://cobot_model/meshes/visual/segment05_visual.stl" scale="0.001 0.001 0.001" />
             </geometry>
             <material name="segment5_material">
@@ -168,5 +168,5 @@
             <origin rpy="0.0 0.0 0.0" xyz="0.0 0.0 0.0" />
             <geometry>
-                <mesh filename="package://cobot_model/meshes/v2_0_hull/segment06_combined.stl" scale="0.001 0.001 0.001" />
+                <mesh filename="package://cobot_model/meshes/visual/segment06_visual.stl" scale="0.001 0.001 0.001" />
             </geometry>
             <material name="segment6_material">
@@ -193,5 +193,5 @@
             </material>
             <geometry>
-                <mesh filename="package://cobot_model/meshes/v2_0_hull/segment07_black.stl" scale="0.001 0.001 0.001" />
+                <mesh filename="package://cobot_model/meshes/visual/segment07_visual.stl" scale="0.001 0.001 0.001" />
             </geometry>
         </visual>
@@ -232,5 +232,5 @@
             </material>
             <geometry>
-                <mesh filename="package://cobot_model/meshes/v2_0_hull/finger01.stl" scale="0.000001 0.000001 0.000001" />
+                <mesh filename="package://cobot_model/meshes/visual/finger01_visual.stl" scale="0.000001 0.000001 0.000001" />
             </geometry>
         </visual>
@@ -254,5 +254,5 @@
             </material>
             <geometry>
-                <mesh filename="package://cobot_model/meshes/v2_0_hull/finger02.stl" scale="0.000001 0.000001 0.000001" />
+                <mesh filename="package://cobot_model/meshes/visual/finger02_visual.stl" scale="0.000001 0.000001 0.000001" />
             </geometry>
         </visual>

Commit message: fix TCP link in urdf and re-order entries in srdf

File: src/cobot_model/urdf/robot_model.urdf.xacro (robot description, xacro)
@@ -204,5 +204,5 @@
         <inertial>
             <mass value="0.2" />
-            <origin rpy="0.0 0.0 0.0" xyz="0.0 0.0 0.0" />
+            <origin rpy="0.0 0.0 0.0" xyz="0.0 0.0 0.02" />
             <inertia ixx="0.00040667" iyy="0.00030104" izz="0.00059971" ixy="0.0" ixz="0.0" iyz="0.0" />
         </inertial>
@@ -221,5 +221,5 @@
             <origin rpy="0.0 0.0 0.0" xyz="0.0 0.0 0.0" />
             <geometry>
-                <cylinder radius="0.0001" length="0.0001" />
+                <cylinder radius="0.00001" length="0.00001" />
             </geometry>
         </collision>
@@ -243,5 +243,5 @@
         <inertial>
             <mass value="0.05" />
-            <origin rpy="0.0 0.0 0.0" xyz="0.0 0.0 0.0" />
+            <origin rpy="0.0 0.0 0.0" xyz="0.0 -0.03 -0.03" />
             <inertia ixx="3.46666667e-05" iyy="2.64166667e-05" izz="1.78833333e-05" ixy="0.0" ixz="0.0" iyz="0.0" />
         </inertial>
@@ -265,5 +265,5 @@
         <inertial>
             <mass value="0.05" />
-            <origin rpy="0.0 0.0 0.0" xyz="0.0 0.0 0.0" />
+            <origin rpy="0.0 0.0 0.0" xyz="0.0 0.03 -0.03" />
             <inertia ixx="3.46666667e-05" iyy="2.64166667e-05" izz="1.78833333e-05" ixy="0.0" ixz="0.0" iyz="0.0" />
         </inertial>
@@ -323,13 +323,13 @@
     </joint>
     <joint name="joint_6" type="revolute">
-        <origin rpy="0.0 -1.570 0.0" xyz="0.26 0.0 -0.041" />
+        <origin rpy="0.0 1.570 0.0" xyz="0.22 0.0 -0.041" />
         <parent link="segment6" />
         <child link="segment7" />
         <axis xyz="0 0 1" />
-        <limit effort="20." velocity="3.141593" lower="-2.356194" upper="2.356194" />
+        <limit effort="20." velocity="3.141593" lower="-3.14" upper="3.14" />
         <dynamics damping="0.0" friction="0.0" />
     </joint>
     <joint name="JFix_TCP" type="fixed">
-        <origin rpy="0.0 3.141593 0.0" xyz="0.0 0.0 -0.06" />
+        <origin rpy="0.0 0.0 0.0" xyz="0.0 0.0 -0.01"/>
         <parent link="segment7" />
         <child link="TCP" />
@@ -341,5 +341,5 @@
     </joint>
     <joint name="finger1_joint" type="prismatic">
-        <origin rpy="0.0 0.0 0.0" xyz="0.0 0.0 0.0" />
+        <origin rpy="0.0 0.0 0.0" xyz="0.0 0.0 0.1" />
         <parent link="TCP" />
         <child link="finger1" />
@@ -348,5 +348,5 @@
     </joint>
     <joint name="finger2_joint" type="prismatic">
-        <origin rpy="0.0 0.0 0.0" xyz="0.0 0.0 0.0" />
+        <origin rpy="0.0 0.0 0.0" xyz="0.0 0.0 0.1" />
         <parent link="TCP" />
         <child link="finger2" />
