Commit message: update model to match real cobot

File: src/cobot_model/urdf/robot_model.urdf.xacro (robot description, xacro)
@@ -146,5 +146,5 @@
             <origin rpy="0.0 0.0 0.0" xyz="0.0 0.0 0.0" />
             <geometry>
-                <mesh filename="package://cobot_model/meshes/visual/segment05_visual.stl" scale="0.001 0.001 0.001" />
+                <mesh filename="package://cobot_model/meshes/visual/segment05_visual_big.stl" scale="0.001 0.001 0.001" />
             </geometry>
             <material name="segment5_material">
@@ -155,5 +155,5 @@
             <origin rpy="0.0 0.0 0.0" xyz="0.0 0.0 0.0" />
             <geometry>
-                <mesh filename="package://cobot_model/meshes/collision/segment05_collision.stl" scale="0.001 0.001 0.001" />
+                <mesh filename="package://cobot_model/meshes/collision/segment05_collision_big.stl" scale="0.001 0.001 0.001" />
             </geometry>
         </collision>
@@ -161,5 +161,5 @@
             <mass value="1.1" />
             <origin rpy="0.0 0.0 0.0" xyz="0.0 0.0 0.071" />
-            <inertia ixx="0.00326077" iyy="0.00326077" izz="0.00277255" ixy="0.0" ixz="0.0" iyz="0.0" />
+            <inertia ixx="0.00623544" iyy="0.00623544" izz="0.00277255" ixy="0.0" ixz="0.0" iyz="0.0" />
         </inertial>
     </link>
@@ -168,5 +168,5 @@
             <origin rpy="0.0 0.0 0.0" xyz="0.0 0.0 0.0" />
             <geometry>
-                <mesh filename="package://cobot_model/meshes/visual/segment06_visual.stl" scale="0.001 0.001 0.001" />
+                <mesh filename="package://cobot_model/meshes/visual/segment06_visual_small.stl" scale="0.001 0.001 0.001" />
             </geometry>
             <material name="segment6_material">
@@ -177,35 +177,35 @@
             <origin rpy="0.0 0.0 0.0" xyz="0.0 0.0 0.0" />
             <geometry>
-                <mesh filename="package://cobot_model/meshes/collision/segment06_collision.stl" scale="0.001 0.001 0.001" />
+                <mesh filename="package://cobot_model/meshes/collision/segment06_collision_small.stl" scale="0.001 0.001 0.001" />
             </geometry>
         </collision>
         <inertial>
             <mass value="1.5" />
-            <origin rpy="0.0 0.0 0.0" xyz="0.12 0.0 0.0" />
-            <inertia ixx="0.00319363" iyy="0.01012625" izz="0.01115763" ixy="0.0" ixz="0.0" iyz="0.0" />
-        </inertial>
-    </link>
-    <link name="segment7">
-        <visual>
-            <origin rpy="0.0 0.0 0.0" xyz="0.0 0.0 0.0" />
+            <origin rpy="0.0 0.0 0.0" xyz="0.10 0.0 0.0" />
+            <inertia ixx="0.00319363" iyy="0.00513113" izz="0.0061625" ixy="0.0" ixz="0.0" iyz="0.0" />
+        </inertial>
+    </link>
+      <link name="segment7">
+        <visual>
+            <origin rpy="0.0 0.0 0.0" xyz="0.0 -0.01 -0.03"/>
             <material name="Aterul">
-                <color rgba="0.0 0.0 0.0 1.0" />
-            </material>
-            <geometry>
-                <mesh filename="package://cobot_model/meshes/visual/segment07_visual.stl" scale="0.001 0.001 0.001" />
-            </geometry>
-        </visual>
-        <collision>
-            <origin rpy="0.0 0.0 0.0" xyz="0.0 0.0 0.0" />
-            <geometry>
-                <mesh filename="package://cobot_model/meshes/collision/segment07_collision.stl" scale="0.001 0.001 0.001" />
-            </geometry>
-        </collision>
-        <inertial>
-            <mass value="0.2" />
-            <origin rpy="0.0 0.0 0.0" xyz="0.0 0.0 0.02" />
-            <inertia ixx="0.00040667" iyy="0.00030104" izz="0.00059971" ixy="0.0" ixz="0.0" iyz="0.0" />
-        </inertial>
-    </link>
+                <color rgba="0.0 0.0 0.0 1.0"/>
+            </material>
+            <geometry>
+            <cylinder radius="0.01" length="0.16"/>
+            </geometry>
+        </visual>
+        <collision>
+            <origin rpy="0.0 0.0 0.0" xyz="0.0 -0.05 0.0"/>
+            <geometry>
+            <box size="0.10 0.10 0.15" />
+            </geometry>
+        </collision>
+        <inertial>
+            <mass value="1.5"/>
+            <origin rpy="0.0 0.0 0.0" xyz="0.0 0.0 0.0"/>
+            <inertia ixx="0.0025" ixy="0.0" ixz="0.0" iyy="0.0040625" iyz="0.0" izz="0.0040625"/>
+        </inertial>
+  </link>
     <link name="TCP">
         <visual>
@@ -295,5 +295,5 @@
         <child link="segment3" />
         <axis xyz="0 0 1" />
-        <limit effort="150.0" velocity="3.141593" lower="-1.570796" upper="1.570796" />
+        <limit effort="150.0" velocity="3.141593" lower="-0.9" upper="1.570796" />
         <dynamics damping="0.0" friction="0.0" />
     </joint>
@@ -315,5 +315,5 @@
     </joint>
     <joint name="joint_5" type="revolute">
-        <origin rpy="-1.570 -1.570 0.0" xyz="0.0 0.042 0.103" />
+        <origin rpy="-1.570 -1.570 0.0" xyz="0.0 0.042 0.193" />
         <parent link="segment5" />
         <child link="segment6" />
@@ -323,15 +323,15 @@
     </joint>
     <joint name="joint_6" type="revolute">
-        <origin rpy="0.0 1.570 0.0" xyz="0.22 0.0 -0.041" />
-        <parent link="segment6" />
-        <child link="segment7" />
-        <axis xyz="0 0 1" />
-        <limit effort="20." velocity="3.141593" lower="-3.14" upper="3.14" />
-        <dynamics damping="0.0" friction="0.0" />
+        <origin rpy="0.0 1.57 -0.785" xyz="0.2 -0.04 -0.041"/>
+        <parent link="segment6"/>
+        <child link="segment7"/>
+        <axis xyz="0 0 1"/>
+        <limit effort="20." lower="-2.356194" upper="2.356194" velocity="3.141593"/>
+        <dynamics damping="0.0" friction="0.0"/>
     </joint>
     <joint name="JFix_TCP" type="fixed">
-        <origin rpy="0.0 0.0 0.0" xyz="0.0 0.0 -0.01"/>
-        <parent link="segment7" />
-        <child link="TCP" />
+        <origin rpy="-1.57 1.57 0.0" xyz="0.0 -0.04 0.0"/>
+        <parent link="segment7"/>
+        <child link="TCP"/>
     </joint>
    <joint name="JFix_Base" type="fixed">

Commit message: new gripper added + segment 6 re-modelled

File: src/cobot_model/urdf/robot_model.urdf.xacro (robot description, xacro)
@@ -182,5 +182,5 @@
         <inertial>
             <mass value="1.5" />
-            <origin rpy="0.0 0.0 0.0" xyz="0.10 0.0 0.0" />
+            <origin rpy="0.0 0.0 0.0" xyz="0.05 0.0 0.0" />
             <inertia ixx="0.00319363" iyy="0.00513113" izz="0.0061625" ixy="0.0" ixz="0.0" iyz="0.0" />
         </inertial>
@@ -188,22 +188,22 @@
       <link name="segment7">
         <visual>
-            <origin rpy="0.0 0.0 0.0" xyz="0.0 -0.01 -0.03"/>
+            <origin rpy="0.0 0.0 0.0" xyz="0.0 0.0 0.0"/>
             <material name="Aterul">
                 <color rgba="0.0 0.0 0.0 1.0"/>
             </material>
             <geometry>
-            <cylinder radius="0.01" length="0.16"/>
-            </geometry>
-        </visual>
-        <collision>
-            <origin rpy="0.0 0.0 0.0" xyz="0.0 -0.05 0.0"/>
-            <geometry>
-            <box size="0.10 0.10 0.15" />
-            </geometry>
-        </collision>
-        <inertial>
-            <mass value="1.5"/>
+                <mesh filename="package://cobot_model/meshes/visual/gripper_frame_visual.stl" scale="0.001 0.001 0.001"/>
+            </geometry>
+        </visual>
+        <collision>
             <origin rpy="0.0 0.0 0.0" xyz="0.0 0.0 0.0"/>
-            <inertia ixx="0.0025" ixy="0.0" ixz="0.0" iyy="0.0040625" iyz="0.0" izz="0.0040625"/>
+            <geometry>
+                <mesh filename="package://cobot_model/meshes/collision/gripper_frame_collision.stl" scale="0.001 0.001 0.001"/>
+            </geometry>
+        </collision>
+        <inertial>
+            <mass value="3.0"/>
+            <origin rpy="0.0 0.0 0.0" xyz="0.0 0.0 0.07"/>
+            <inertia ixx="0.00910541" iyy="0.01309269" izz="0.01268213" ixy="0.0" ixz="0.0" iyz="0.0" />
         </inertial>
   </link>
@@ -219,5 +219,5 @@
         </visual>
         <collision>
-            <origin rpy="0.0 0.0 0.0" xyz="0.0 0.0 0.0" />
+            <origin rpy="0.0 0.0 0.0" xyz="-0.12 -0.03 0.0"/>
             <geometry>
                 <cylinder radius="0.00001" length="0.00001" />
@@ -227,21 +227,21 @@
     <link name="finger1">
         <visual>
-            <origin rpy="0.0 0.0 0.0" xyz="0.0 0.0 0.0" />
+           <origin rpy="0.0 0.0 0.0" xyz="0.0 0.01 -0.08"/>
             <material name="silver">
                 <color rgba="0.629 0.629 0.625 1.0" />
             </material>
             <geometry>
-                <mesh filename="package://cobot_model/meshes/visual/finger01_visual.stl" scale="0.000001 0.000001 0.000001" />
-            </geometry>
-        </visual>
-        <collision>
-            <origin rpy="0.0 0.0 0.0" xyz="0.0 0.0 0.0" />
-            <geometry>
-                <mesh filename="package://cobot_model/meshes/collision/finger01_collision.stl" scale="0.000001 0.000001 0.000001" />
+                <mesh filename="package://cobot_model/meshes/visual/finger01_real_visual.stl" scale="0.001 0.001 0.001" />
+            </geometry>
+        </visual>
+        <collision>
+            <origin rpy="0.0 0.0 0.0" xyz="0.0 0.01 -0.08"/>
+            <geometry>
+                <mesh filename="package://cobot_model/meshes/collision/finger01_real_collision.stl" scale="0.001 0.001 0.001" />
             </geometry>
         </collision>
         <inertial>
             <mass value="0.05" />
-            <origin rpy="0.0 0.0 0.0" xyz="0.0 -0.03 -0.03" />
+            <origin rpy="-0.785 0.0 0.0" xyz="0.02 0.03 0.03" />
             <inertia ixx="3.46666667e-05" iyy="2.64166667e-05" izz="1.78833333e-05" ixy="0.0" ixz="0.0" iyz="0.0" />
         </inertial>
@@ -249,21 +249,21 @@
     <link name="finger2">
         <visual>
-            <origin rpy="0.0 0.0 0.0" xyz="0.0 0.0 0.0" />
+            <origin rpy="0.0 0.0 0.0" xyz="0.0 0.01 -0.08"/>
             <material name="silver">
                 <color rgba="0.629 0.629 0.625 1.0" />
             </material>
             <geometry>
-                <mesh filename="package://cobot_model/meshes/visual/finger02_visual.stl" scale="0.000001 0.000001 0.000001" />
-            </geometry>
-        </visual>
-        <collision>
-            <origin rpy="0.0 0.0 0.0" xyz="0.0 0.0 0.0" />
-            <geometry>
-                <mesh filename="package://cobot_model/meshes/collision/finger02_collision.stl" scale="0.000001 0.000001 0.000001" />
+                <mesh filename="package://cobot_model/meshes/visual/finger02_real_visual.stl" scale="0.001 0.001 0.001" />
+            </geometry>
+        </visual>
+        <collision>
+            <origin rpy="0.0 0.0 0.0" xyz="0.0 0.01 -0.08"/>
+            <geometry>
+                <mesh filename="package://cobot_model/meshes/collision/finger02_real_collision.stl" scale="0.001 0.001 0.001" />
             </geometry>
         </collision>
         <inertial>
             <mass value="0.05" />
-            <origin rpy="0.0 0.0 0.0" xyz="0.0 0.03 -0.03" />
+            <origin rpy="-0.785 0.0 0.0" xyz="-0.02 0.03 0.03" />
             <inertia ixx="3.46666667e-05" iyy="2.64166667e-05" izz="1.78833333e-05" ixy="0.0" ixz="0.0" iyz="0.0" />
         </inertial>
@@ -323,5 +323,5 @@
     </joint>
     <joint name="joint_6" type="revolute">
-        <origin rpy="0.0 1.57 -0.785" xyz="0.2 -0.04 -0.041"/>
+        <origin rpy="0.0 1.57 0.0" xyz="0.14 0.0 -0.04"/>
         <parent link="segment6"/>
         <child link="segment7"/>
@@ -331,5 +331,5 @@
     </joint>
     <joint name="JFix_TCP" type="fixed">
-        <origin rpy="-1.57 1.57 0.0" xyz="0.0 -0.04 0.0"/>
+        <origin rpy="-0.785 0.0 0.0" xyz="0.0 -0.01 0.08"/>
         <parent link="segment7"/>
         <child link="TCP"/>
@@ -341,15 +341,15 @@
     </joint>
     <joint name="finger1_joint" type="prismatic">
-        <origin rpy="0.0 0.0 0.0" xyz="0.0 0.0 0.1" />
+        <origin rpy="0.785 0.0 0.0" xyz="0.0 0.0 0.0" />
         <parent link="TCP" />
         <child link="finger1" />
-        <axis xyz="0 -1 0" />
+        <axis xyz="-1 0 0" />
         <limit effort="30.0" velocity="0.1" lower="-0.01" upper="0.015" />
     </joint>
     <joint name="finger2_joint" type="prismatic">
-        <origin rpy="0.0 0.0 0.0" xyz="0.0 0.0 0.1" />
+        <origin rpy="0.785 0.0 0.0" xyz="0.0 0.0 0.0" />
         <parent link="TCP" />
         <child link="finger2" />
-        <axis xyz="0 1 0" />
+        <axis xyz="1 0 0" />
         <limit effort="30.0" velocity="0.1" lower="-0.01" upper="0.015" />
         <mimic joint="finger1_joint" />

Commit message: real gripper added

File: src/cobot_model/urdf/robot_model.urdf.xacro (robot description, xacro)
@@ -190,8 +190,8 @@
             <origin rpy="0.0 0.0 0.0" xyz="0.0 0.0 0.0"/>
             <material name="Aterul">
-                <color rgba="0.0 0.0 0.0 1.0"/>
-            </material>
-            <geometry>
-                <mesh filename="package://cobot_model/meshes/visual/gripper_frame_visual.stl" scale="0.001 0.001 0.001"/>
+                <color rgba="1.0 1.0 1.0 1.0"/>
+            </material>
+            <geometry>
+                <mesh filename="package://cobot_model/meshes/visual/segment07_real_visual.stl" scale="0.001 0.001 0.001"/>
             </geometry>
         </visual>
@@ -199,11 +199,11 @@
             <origin rpy="0.0 0.0 0.0" xyz="0.0 0.0 0.0"/>
             <geometry>
-                <mesh filename="package://cobot_model/meshes/collision/gripper_frame_collision.stl" scale="0.001 0.001 0.001"/>
-            </geometry>
-        </collision>
-        <inertial>
-            <mass value="3.0"/>
-            <origin rpy="0.0 0.0 0.0" xyz="0.0 0.0 0.07"/>
-            <inertia ixx="0.00910541" iyy="0.01309269" izz="0.01268213" ixy="0.0" ixz="0.0" iyz="0.0" />
+                <mesh filename="package://cobot_model/meshes/collision/segment07_real_collision.stl" scale="0.001 0.001 0.001"/>
+            </geometry>
+        </collision>
+        <inertial>
+            <mass value="4.0"/>
+            <origin rpy="0.0 0.0 0.0" xyz="0.0 -0.09 0.04"/>
+           <inertia ixx="0.02693367" iyy="0.01533367" izz="0.02185067" ixy="0.0" ixz="0.0" iyz="0.0" />
         </inertial>
   </link>
@@ -227,5 +227,5 @@
     <link name="finger1">
         <visual>
-           <origin rpy="0.0 0.0 0.0" xyz="0.0 0.01 -0.08"/>
+           <origin rpy="0.0 0.0 0.0" xyz="0.0 0.08 -0.06"/>
             <material name="silver">
                 <color rgba="0.629 0.629 0.625 1.0" />
@@ -236,5 +236,5 @@
         </visual>
         <collision>
-            <origin rpy="0.0 0.0 0.0" xyz="0.0 0.01 -0.08"/>
+            <origin rpy="0.0 0.0 0.0" xyz="0.0 0.08 -0.06"/>
             <geometry>
                 <mesh filename="package://cobot_model/meshes/collision/finger01_real_collision.stl" scale="0.001 0.001 0.001" />
@@ -249,5 +249,5 @@
     <link name="finger2">
         <visual>
-            <origin rpy="0.0 0.0 0.0" xyz="0.0 0.01 -0.08"/>
+            <origin rpy="0.0 0.0 0.0" xyz="0.0 0.08 -0.06"/>
             <material name="silver">
                 <color rgba="0.629 0.629 0.625 1.0" />
@@ -258,5 +258,5 @@
         </visual>
         <collision>
-            <origin rpy="0.0 0.0 0.0" xyz="0.0 0.01 -0.08"/>
+            <origin rpy="0.0 0.0 0.0" xyz="0.0 0.08 -0.06"/>
             <geometry>
                 <mesh filename="package://cobot_model/meshes/collision/finger02_real_collision.stl" scale="0.001 0.001 0.001" />
@@ -323,5 +323,5 @@
     </joint>
     <joint name="joint_6" type="revolute">
-        <origin rpy="0.0 1.57 0.0" xyz="0.14 0.0 -0.04"/>
+        <origin rpy="0.0 1.57 0.0" xyz="0.156 0.0 -0.04"/>
         <parent link="segment6"/>
         <child link="segment7"/>
@@ -331,5 +331,5 @@
     </joint>
     <joint name="JFix_TCP" type="fixed">
-        <origin rpy="-0.785 0.0 0.0" xyz="0.0 -0.01 0.08"/>
+        <origin rpy="-0.785 0.0 0.0" xyz="0.0 -0.08 0.06"/>
         <parent link="segment7"/>
         <child link="TCP"/>

Commit message: re-modelled segment 5 and 6

File: src/cobot_model/urdf/robot_model.urdf.xacro (robot description, xacro)
@@ -146,5 +146,5 @@
             <origin rpy="0.0 0.0 0.0" xyz="0.0 0.0 0.0" />
             <geometry>
-                <mesh filename="package://cobot_model/meshes/visual/segment05_visual_big.stl" scale="0.001 0.001 0.001" />
+                <mesh filename="package://cobot_model/meshes/visual/segment05_power_visual.stl" scale="0.001 0.001 0.001" />
             </geometry>
             <material name="segment5_material">
@@ -155,5 +155,5 @@
             <origin rpy="0.0 0.0 0.0" xyz="0.0 0.0 0.0" />
             <geometry>
-                <mesh filename="package://cobot_model/meshes/collision/segment05_collision_big.stl" scale="0.001 0.001 0.001" />
+                <mesh filename="package://cobot_model/meshes/collision/segment05_power_collision.stl" scale="0.001 0.001 0.001" />
             </geometry>
         </collision>
@@ -168,5 +168,5 @@
             <origin rpy="0.0 0.0 0.0" xyz="0.0 0.0 0.0" />
             <geometry>
-                <mesh filename="package://cobot_model/meshes/visual/segment06_visual_small.stl" scale="0.001 0.001 0.001" />
+                <mesh filename="package://cobot_model/meshes/visual/segment06_power_visual.stl" scale="0.001 0.001 0.001" />
             </geometry>
             <material name="segment6_material">
@@ -177,5 +177,5 @@
             <origin rpy="0.0 0.0 0.0" xyz="0.0 0.0 0.0" />
             <geometry>
-                <mesh filename="package://cobot_model/meshes/collision/segment06_collision_small.stl" scale="0.001 0.001 0.001" />
+                <mesh filename="package://cobot_model/meshes/collision/segment06_power_collision.stl" scale="0.001 0.001 0.001" />
             </geometry>
         </collision>
@@ -307,5 +307,5 @@
     </joint>
     <joint name="joint_4" type="revolute">
-        <origin rpy="-1.5708 0.0 -1.5708" xyz="0.024 0.0 -0.168" />
+        <origin rpy="-1.5708 0.0 -1.5708" xyz="0.062 0.0 -0.168"/>
         <parent link="segment4" />
         <child link="segment5" />

Commit message: align joint init positions and joint limits with real cobot

File: src/cobot_model/urdf/robot_model.urdf.xacro (robot description, xacro)
@@ -283,25 +283,25 @@
     </joint>
     <joint name="joint_1" type="revolute">
-        <origin rpy="0.0 0.0 0.0" xyz="0.0 0.0 0.0" />
+        <origin rpy="0.0 0.0 -3.14" xyz="0.0 0.0 0.0" />
         <parent link="segment1" />
         <child link="segment2" />
         <axis xyz="0 0 1" />
-        <limit effort="200.0" velocity="3.141593" lower="-0.7853976732051033" upper="3.9269903267948965" />
+        <limit effort="200.0" velocity="3.141593" lower="-2.37365" upper="2.37365" />
         <dynamics damping="0.0" friction="0.0" />
     </joint>
     <joint name="joint_2" type="revolute">
-        <origin rpy="1.5708 0.0 0.0" xyz="0.0 -0.111 0.118" />
+        <origin rpy="1.5708 -1.5708 0.0" xyz="0.0 -0.111 0.118" />
         <parent link="segment2" />
         <child link="segment3" />
         <axis xyz="0 0 1" />
-        <limit effort="150.0" velocity="3.141593" lower="-0.9" upper="2.35" />
+        <limit effort="150.0" velocity="3.141593" lower="-2.26893" upper="0.785398" />
         <dynamics damping="0.0" friction="0.0" />
     </joint>
     <joint name="joint_3" type="revolute">
-        <origin rpy="0.0 0.0 0.0" xyz="0.254 0.0 0.06" />
+        <origin rpy="0.0 0.0 -1.57" xyz="0.254 0.0 0.06" />
         <parent link="segment3" />
         <child link="segment4" />
         <axis xyz="0 0 1" />
-        <limit effort="100.0" velocity="3.141593" lower="-2.35" upper="1.570796" />
+        <limit effort="100.0" velocity="3.141593" lower="-0.785398" upper="2.26893" />
         <dynamics damping="0.0" friction="0.0" />
     </joint>
@@ -315,5 +315,5 @@
     </joint>
     <joint name="joint_5" type="revolute">
-        <origin rpy="-1.570 -1.570 0.0" xyz="0.0 0.042 0.193" />
+        <origin rpy="-1.570 -1.570 0.0" xyz="0.0 0.042 0.183" />
         <parent link="segment5" />
         <child link="segment6" />
@@ -327,5 +327,5 @@
         <child link="segment7"/>
         <axis xyz="0 0 1"/>
-        <limit effort="20." lower="-3.1" upper="3.1" velocity="3.141593"/>
+        <limit effort="20." lower="-2.37365" upper="2.37365" velocity="3.141593"/>
         <dynamics damping="0.0" friction="0.0"/>
     </joint>

Commit message: real carriage mesh added / joint position and limits updated

File: src/cobot_model/urdf/robot_model.urdf.xacro (robot description, xacro)
@@ -36,5 +36,5 @@
              <origin rpy="0.0 0.0 0.0" xyz="0.0 0.0 0.0" />
             <geometry>
-                <mesh filename="package://cobot_model/meshes/visual/carriage_visual.dae" scale="0.001 0.001 0.001" />
+                <mesh filename="package://cobot_model/meshes/visual/carriage_real_visual.dae" scale="0.001 0.001 0.001" />
                 <material name="silver">
                     <color rgba="1.0 1.0 1.0 1.0" />
@@ -45,5 +45,5 @@
              <origin rpy="0.0 0.0 0.0" xyz="0.0 0.0 0.0" />
             <geometry>
-                <mesh filename="package://cobot_model/meshes/collision/carriage_collision.dae" scale="0.001 0.001 0.001" />
+                <mesh filename="package://cobot_model/meshes/collision/carriage_real_collision.stl" scale="0.001 0.001 0.001" />
             </geometry>
         </collision>
@@ -271,12 +271,12 @@
     <!-- Joints -->
     <joint name="joint_0" type="prismatic">
-        <origin rpy="0.0 0.0 0.0" xyz="0.0 0.0 0.3" />
+        <origin rpy="0.0 0.0 0.0" xyz="0.0 0.0 0.0" />
         <parent link="lin_axis" />
         <child link="lin_axis_carriage" />
         <axis xyz="0 0 1" />
-        <limit effort="300.0" velocity="3.141593" lower="-.29" upper=".55" />
+        <limit effort="300.0" velocity="3.141593" lower="0.0" upper="0.894" />
     </joint>
     <joint name="mount_fixture" type="fixed">
-        <origin rpy="0.0 0.0 0.0" xyz="0.0 0.3 0.3" />
+        <origin rpy="0.0 0.0 0.0" xyz="0.0 0.37 0.52" />
         <parent link="lin_axis_carriage" />
         <child link="segment1" />

Commit message: updated carriage mesh + corresponding joint limit

File: src/cobot_model/urdf/robot_model.urdf.xacro (robot description, xacro)
@@ -275,5 +275,5 @@
         <child link="lin_axis_carriage" />
         <axis xyz="0 0 1" />
-        <limit effort="300.0" velocity="3.141593" lower="0.0" upper="0.894" />
+        <limit effort="300.0" velocity="3.141593" lower="-0.0001" upper="0.894" />
     </joint>
     <joint name="mount_fixture" type="fixed">
