Commit message: enable usage of simple geometric objects for collisions

File: src/cobot_model/urdf/robot_model.urdf.xacro (robot description, xacro)
@@ -1,4 +1,5 @@
 <?xml version="1.0" ?>
 <robot xmlns:xacro="http://www.ros.org/wiki/xacro">
+    <xacro:arg name="use_collision_meshes" default="true" />
     <link name="world" />
     <joint name="robot_in_world" type="fixed">
@@ -21,8 +22,16 @@
         </visual>
         <collision>
-            <origin rpy="0.0 0.0 0.0" xyz="0.0 0.0 0.0" />
-            <geometry>
-                <mesh filename="package://cobot_model/meshes/collision/axis_collision.dae" scale="0.001 0.001 0.001" />
-            </geometry>
+            <xacro:if value="${'$(arg use_collision_meshes)' == 'true'}">
+                <origin rpy="0.0 0.0 0.0" xyz="0.0 0.0 0.0" />
+                <geometry>
+                    <mesh filename="package://cobot_model/meshes/collision/axis_collision.dae" scale="0.001 0.001 0.001" />
+                </geometry>
+            </xacro:if>
+            <xacro:unless value="${'$(arg use_collision_meshes)' == 'true'}">
+                <origin rpy="0.0 0.0 0.0" xyz="0.0 0.03 0.6"/>
+                <geometry>
+                    <box size="0.162 0.069 1.21"/>
+                </geometry>
+            </xacro:unless>
         </collision>
         <inertial>
@@ -43,8 +52,16 @@
         </visual>
         <collision>
-             <origin rpy="0.0 0.0 0.0" xyz="0.0 0.0 0.0" />
-            <geometry>
-                <mesh filename="package://cobot_model/meshes/collision/carriage_real_collision.stl" scale="0.001 0.001 0.001" />
-            </geometry>
+            <xacro:if value="${'$(arg use_collision_meshes)' == 'true'}">
+                <origin rpy="0.0 0.0 0.0" xyz="0.0 0.0 0.0" />
+                <geometry>
+                   <mesh filename="package://cobot_model/meshes/visual/carriage_real_visual.dae" scale="0.001 0.001 0.001" />
+                </geometry>
+            </xacro:if>
+            <xacro:unless value="${'$(arg use_collision_meshes)' == 'true'}">
+                <origin rpy="0.0 0.0 0.0" xyz="0.06 0.26 0.2"/>
+                <geometry>
+                    <box size="0.302 0.431 0.02"/>
+                </geometry>
+            </xacro:unless>
         </collision>
         <inertial>
@@ -65,8 +82,16 @@
         </visual>
         <collision>
-            <origin rpy="0.0 0.0 0.0" xyz="0.0 0.0 0.0" />
-            <geometry>
-                <mesh filename="package://cobot_model/meshes/collision/segment01_collision.stl" scale="0.001 0.001 0.001" />
-            </geometry>
+            <xacro:if value="${'$(arg use_collision_meshes)' == 'true'}">
+                <origin rpy="0.0 0.0 0.0" xyz="0.0 0.0 0.0" />
+                <geometry>
+                    <mesh filename="package://cobot_model/meshes/collision/segment01_collision.stl" scale="0.001 0.001 0.001" />
+                </geometry>
+            </xacro:if>
+            <xacro:unless value="${'$(arg use_collision_meshes)' == 'true'}">
+            <origin rpy="0.0 0.0 0.0" xyz="0.0 0.0 -0.156"/>
+                <geometry>
+                    <cylinder radius="0.09" length="0.312"/>
+                </geometry>
+            </xacro:unless>
         </collision>
         <inertial>
@@ -87,8 +112,16 @@
         </visual>
         <collision>
-            <origin rpy="0.0 0.0 0.0" xyz="0.0 0.0 0.0" />
-            <geometry>
-                <mesh filename="package://cobot_model/meshes/collision/segment02_collision.stl" scale="0.001 0.001 0.001" />
-            </geometry>
+            <xacro:if value="${'$(arg use_collision_meshes)' == 'true'}">
+                <origin rpy="0.0 0.0 0.0" xyz="0.0 0.0 0.0" />
+                <geometry>
+                    <mesh filename="package://cobot_model/meshes/collision/segment02_collision.stl" scale="0.001 0.001 0.001" />
+                </geometry>
+            </xacro:if>
+            <xacro:unless value="${'$(arg use_collision_meshes)' == 'true'}">
+                <origin rpy="0.0 0.0 0.0" xyz="0.0 0.0 0.09"/>
+                <geometry>
+                    <box size="0.155 0.238 0.186"/>
+                </geometry>
+            </xacro:unless>
         </collision>
         <inertial>
@@ -109,8 +142,16 @@
         </visual>
         <collision>
-            <origin rpy="0.0 0.0 0.0" xyz="0.0 0.0 0.0" />
-            <geometry>
-                <mesh filename="package://cobot_model/meshes/collision/segment03_collision.stl" scale="0.001 0.001 0.001" />
-            </geometry>
+            <xacro:if value="${'$(arg use_collision_meshes)' == 'true'}">
+                <origin rpy="0.0 0.0 0.0" xyz="0.0 0.0 0.0" />
+                <geometry>
+                    <mesh filename="package://cobot_model/meshes/collision/segment03_collision.stl" scale="0.001 0.001 0.001" />
+                </geometry>
+            </xacro:if>
+            <xacro:unless value="${'$(arg use_collision_meshes)' == 'true'}">
+                <origin rpy="0.0 1.57 0.0" xyz="0.126 0.0 0.06"/>
+                <geometry>
+                    <cylinder radius="0.06" length="0.372"/>
+                </geometry>
+            </xacro:unless>
         </collision>
         <inertial>
@@ -131,8 +172,16 @@
         </visual>
         <collision>
-             <origin rpy="0.0 0.0 0.0" xyz="0.0 0.0 0.0" />
-            <geometry>
-                <mesh filename="package://cobot_model/meshes/collision/segment04_collision.stl" scale="0.001 0.001 0.001" />
-            </geometry>
+            <xacro:if value="${'$(arg use_collision_meshes)' == 'true'}">
+                <origin rpy="0.0 0.0 0.0" xyz="0.0 0.0 0.0" />
+                <geometry>
+                    <mesh filename="package://cobot_model/meshes/collision/segment04_collision.stl" scale="0.001 0.001 0.001" />
+                </geometry>
+            </xacro:if>
+            <xacro:unless value="${'$(arg use_collision_meshes)' == 'true'}">
+                <origin rpy="0.0 0.0 0.0" xyz="0.0 0.0 -0.1125"/>
+                <geometry>
+                    <cylinder radius="0.07" length="0.225"/>
+                </geometry>
+            </xacro:unless>
         </collision>
         <inertial>
@@ -153,8 +202,16 @@
         </visual>
         <collision>
-            <origin rpy="0.0 0.0 0.0" xyz="0.0 0.0 0.0" />
-            <geometry>
-                <mesh filename="package://cobot_model/meshes/collision/segment05_power_collision.stl" scale="0.001 0.001 0.001" />
-            </geometry>
+            <xacro:if value="${'$(arg use_collision_meshes)' == 'true'}">
+                <origin rpy="0.0 0.0 0.0" xyz="0.0 0.0 0.0" />
+                <geometry>
+                    <mesh filename="package://cobot_model/meshes/collision/segment05_power_collision.stl" scale="0.001 0.001 0.001" />
+                </geometry>
+            </xacro:if>
+            <xacro:unless value="${'$(arg use_collision_meshes)' == 'true'}">
+                <origin rpy="0.0 0.0 0.0" xyz="0.0 0.0 0.1"/>
+                <geometry>
+                    <cylinder radius="0.07" length="0.23"/>
+                </geometry>
+            </xacro:unless>
         </collision>
         <inertial>
@@ -175,8 +232,16 @@
         </visual>
         <collision>
-            <origin rpy="0.0 0.0 0.0" xyz="0.0 0.0 0.0" />
-            <geometry>
-                <mesh filename="package://cobot_model/meshes/collision/segment06_power_collision.stl" scale="0.001 0.001 0.001" />
-            </geometry>
+            <xacro:if value="${'$(arg use_collision_meshes)' == 'true'}">
+                <origin rpy="0.0 0.0 0.0" xyz="0.0 0.0 0.0" />
+                <geometry>
+                    <mesh filename="package://cobot_model/meshes/collision/segment06_power_collision.stl" scale="0.001 0.001 0.001" />
+                </geometry>
+             </xacro:if>
+            <xacro:unless value="${'$(arg use_collision_meshes)' == 'true'}">
+                <origin rpy="0.0 1.57 0.0" xyz="0.12 0.0 -0.04"/>
+                <geometry>
+                    <cylinder length="0.15" radius="0.04"/>
+                </geometry>
+            </xacro:unless>
         </collision>
         <inertial>
@@ -197,8 +262,16 @@
         </visual>
         <collision>
-            <origin rpy="0.0 0.0 0.0" xyz="0.0 0.0 0.0"/>
-            <geometry>
-                <mesh filename="package://cobot_model/meshes/collision/segment07_real_collision.stl" scale="0.001 0.001 0.001"/>
-            </geometry>
+            <xacro:if value="${'$(arg use_collision_meshes)' == 'true'}">
+                <origin rpy="0.0 0.0 0.0" xyz="0.0 0.0 0.0"/>
+                <geometry>
+                    <mesh filename="package://cobot_model/meshes/collision/segment07_real_collision.stl" scale="0.001 0.001 0.001"/>
+                </geometry>
+            </xacro:if>
+            <xacro:unless value="${'$(arg use_collision_meshes)' == 'true'}">
+                <origin rpy="-0.786 0.0 0.0" xyz="0.0 -0.1 0.05"/>
+                <geometry>
+                    <box size="0.124 0.135 0.14"/>
+                </geometry>
+            </xacro:unless>
         </collision>
         <inertial>
@@ -219,5 +292,5 @@
         </visual>
         <collision>
-            <origin rpy="0.0 0.0 0.0" xyz="-0.12 -0.03 0.0"/>
+            <origin rpy="0.0 0.0 0.0" xyz="0.0 0.0 0.0" />
             <geometry>
                 <cylinder radius="0.00001" length="0.00001" />
@@ -236,8 +309,16 @@
         </visual>
         <collision>
-            <origin rpy="0.0 0.0 0.0" xyz="0.0 0.08 -0.06"/>
-            <geometry>
-                <mesh filename="package://cobot_model/meshes/collision/finger01_real_collision.stl" scale="0.001 0.001 0.001" />
-            </geometry>
+            <xacro:if value="${'$(arg use_collision_meshes)' == 'true'}">
+                <origin rpy="0.0 0.0 0.0" xyz="0.0 0.08 -0.06"/>
+                <geometry>
+                    <mesh filename="package://cobot_model/meshes/collision/finger01_real_collision.stl" scale="0.001 0.001 0.001" />
+                </geometry>
+            </xacro:if>
+            <xacro:unless value="${'$(arg use_collision_meshes)' == 'true'}">
+                <origin rpy="-0.786 0.25 0.0" xyz="-0.020 0.040 0.036"/>
+                <geometry>
+                    <cylinder length="0.10" radius="0.01"/>
+                </geometry>
+            </xacro:unless>
         </collision>
         <inertial>
@@ -258,8 +339,16 @@
         </visual>
         <collision>
-            <origin rpy="0.0 0.0 0.0" xyz="0.0 0.08 -0.06"/>
-            <geometry>
-                <mesh filename="package://cobot_model/meshes/collision/finger02_real_collision.stl" scale="0.001 0.001 0.001" />
-            </geometry>
+            <xacro:if value="${'$(arg use_collision_meshes)' == 'true'}">
+                 <origin rpy="0.0 0.0 0.0" xyz="0.0 0.08 -0.06"/>
+                <geometry>
+                    <mesh filename="package://cobot_model/meshes/collision/finger02_real_collision.stl" scale="0.001 0.001 0.001" />
+                </geometry>
+            </xacro:if>
+            <xacro:unless value="${'$(arg use_collision_meshes)' == 'true'}">
+                <origin rpy="-0.786 -0.25 0.0" xyz="0.020 0.040 0.036"/>
+                <geometry>
+                    <cylinder length="0.10" radius="0.01"/>
+                </geometry>
+            </xacro:unless>
         </collision>
         <inertial>

Commit message: move TCP in robot model

File: src/cobot_model/urdf/robot_model.urdf.xacro (robot description, xacro)
@@ -281,27 +281,11 @@
         </inertial>
   </link>
-    <link name="TCP">
-        <visual>
-            <origin rpy="0.0 0.0 0.0" xyz="0.0 0.0 0.0" />
-            <geometry>
-                <cylinder radius="0.00001" length="0.000001" />
-            </geometry>
+    <link name="TCP"/>
+    <link name="finger1">
+        <visual>
+           <origin rpy="0.0 0.0 0.0" xyz="0.0 0.065 -0.065"/>
             <material name="silver">
                 <color rgba="0.629 0.629 0.625 1.0" />
             </material>
-        </visual>
-        <collision>
-            <origin rpy="0.0 0.0 0.0" xyz="0.0 0.0 0.0" />
-            <geometry>
-                <cylinder radius="0.00001" length="0.00001" />
-            </geometry>
-        </collision>
-    </link>
-    <link name="finger1">
-        <visual>
-           <origin rpy="0.0 0.0 0.0" xyz="0.0 0.08 -0.06"/>
-            <material name="silver">
-                <color rgba="0.629 0.629 0.625 1.0" />
-            </material>
             <geometry>
                 <mesh filename="package://cobot_model/meshes/visual/finger01_real_visual.stl" scale="0.001 0.001 0.001" />
@@ -310,5 +294,5 @@
         <collision>
             <xacro:if value="${'$(arg use_collision_meshes)' == 'true'}">
-                <origin rpy="0.0 0.0 0.0" xyz="0.0 0.08 -0.06"/>
+                <origin rpy="0.0 0.0 0.0" xyz="0.0 0.065 -0.065"/>
                 <geometry>
                     <mesh filename="package://cobot_model/meshes/collision/finger01_real_collision.stl" scale="0.001 0.001 0.001" />
@@ -330,5 +314,5 @@
     <link name="finger2">
         <visual>
-            <origin rpy="0.0 0.0 0.0" xyz="0.0 0.08 -0.06"/>
+            <origin rpy="0.0 0.0 0.0" xyz="0.0 0.065 -0.065"/>
             <material name="silver">
                 <color rgba="0.629 0.629 0.625 1.0" />
@@ -340,5 +324,5 @@
         <collision>
             <xacro:if value="${'$(arg use_collision_meshes)' == 'true'}">
-                 <origin rpy="0.0 0.0 0.0" xyz="0.0 0.08 -0.06"/>
+                <origin rpy="0.0 0.0 0.0" xyz="0.0 0.065 -0.065"/>
                 <geometry>
                     <mesh filename="package://cobot_model/meshes/collision/finger02_real_collision.stl" scale="0.001 0.001 0.001" />
@@ -420,5 +404,5 @@
     </joint>
     <joint name="JFix_TCP" type="fixed">
-        <origin rpy="-0.785 0.0 0.0" xyz="0.0 -0.08 0.06"/>
+        <origin rpy="-0.785 0.0 0.0" xyz="0.0 -0.02 0.12"/>
         <parent link="segment7"/>
         <child link="TCP"/>
@@ -430,6 +414,6 @@
     </joint>
     <joint name="finger1_joint" type="prismatic">
-        <origin rpy="0.785 0.0 0.0" xyz="0.0 0.0 0.0" />
-        <parent link="TCP" />
+        <origin rpy="0.0 0.0 0.0" xyz="0.0 -0.065 0.065"/>
+        <parent link="segment7" />
         <child link="finger1" />
         <axis xyz="-1 0 0" />
@@ -437,6 +421,6 @@
     </joint>
     <joint name="finger2_joint" type="prismatic">
-        <origin rpy="0.785 0.0 0.0" xyz="0.0 0.0 0.0" />
-        <parent link="TCP" />
+        <origin rpy="0.0 0.0 0.0" xyz="0.0 -0.065 0.065"/>
+        <parent link="segment7" />
         <child link="finger2" />
         <axis xyz="1 0 0" />

Commit message: added vacuum gripper model

File: src/cobot_model/urdf/robot_model.urdf.xacro (robot description, xacro)
@@ -342,4 +342,64 @@
         </inertial>
     </link>
+    <link name="vacuum_gripper_up">
+    <visual>
+      <origin rpy="0.0 0.0 0.0" xyz="0.0 0.026 -0.103"/>
+      <material name="silver">
+        <color rgba="0.629 0.629 0.625 1.0"/>
+      </material>
+      <geometry>
+        <mesh filename="package://cobot_model/meshes/visual/vacuum_gripper_up_visual.stl" scale="0.001 0.001 0.001"/>
+      </geometry>
+    </visual>
+    <collision>
+    <xacro:if value="${'$(arg use_collision_meshes)' == 'true'}">
+        <origin rpy="0.0 0.0 0.0" xyz="0.0 0.026 -0.103"/>
+        <geometry>
+            <mesh filename="package://cobot_model/meshes/collision/vacuum_gripper_up_collision.stl" scale="0.001 0.001 0.001"/>
+        </geometry>
+    </xacro:if>
+    <xacro:unless value="${'$(arg use_collision_meshes)' == 'true'}">
+        <origin rpy="-0.786 0.0 0.0" xyz="0.0 -0.008 0.042"/>
+        <geometry>
+            <cylinder length="0.10" radius="0.01"/>
+        </geometry>
+    </xacro:unless>
+    </collision>
+    <inertial>
+      <mass value="0.05"/>
+      <origin rpy="-0.785 0.0 0.0" xyz="0.0 0.001 0.052"/>
+      <inertia ixx="3.46666667e-05" ixy="0.0" ixz="0.0" iyy="2.64166667e-05" iyz="0.0" izz="1.78833333e-05"/>
+    </inertial>
+  </link>
+  <link name="vacuum_gripper_down">
+    <visual>
+      <origin rpy="0.0 0.0 0.0" xyz="0.0 0.026 -0.103"/>
+      <material name="silver">
+        <color rgba="0.629 0.629 0.625 1.0"/>
+      </material>
+      <geometry>
+        <mesh filename="package://cobot_model/meshes/visual/vacuum_gripper_down_visual.stl" scale="0.001 0.001 0.001"/>
+      </geometry>
+    </visual>
+    <collision>
+        <xacro:if value="${'$(arg use_collision_meshes)' == 'true'}">
+            <origin rpy="0.0 0.0 0.0" xyz="0.0 0.026 -0.103"/>
+            <geometry>
+                <mesh filename="package://cobot_model/meshes/collision/vacuum_gripper_down_collision.stl" scale="0.001 0.001 0.001"/>
+            </geometry>
+        </xacro:if>
+       <xacro:unless value="${'$(arg use_collision_meshes)' == 'true'}">
+            <origin rpy="-0.786 0.0 0.0" xyz="0.0 0.042 -0.008"/>
+            <geometry>
+                <cylinder length="0.10" radius="0.01"/>
+            </geometry>
+       </xacro:unless>
+    </collision>
+    <inertial>
+      <mass value="0.05"/>
+      <origin rpy="-0.785 0.0 0.0" xyz="0.0 0.052 0.001"/>
+      <inertia ixx="3.46666667e-05" ixy="0.0" ixz="0.0" iyy="2.64166667e-05" iyz="0.0" izz="1.78833333e-05"/>
+    </inertial>
+  </link>
     <!-- Joints -->
     <joint name="joint_0" type="prismatic">
@@ -428,3 +488,18 @@
         <mimic joint="finger1_joint" />
     </joint>
+    <joint name="vacuum_up_joint" type="prismatic">
+        <origin rpy="0.0 0.0 0.0" xyz="0.0 -0.065 0.065"/>
+        <parent link="segment7"/>
+        <child link="vacuum_gripper_up"/>
+        <axis xyz="0 1 1"/>
+        <limit effort="30.0" lower="-0.01" upper="0.035" velocity="0.1"/>
+    </joint>
+    <joint name="vacuum_down_joint" type="prismatic">
+        <origin rpy="0.0 0.0 0.0" xyz="0.0 -0.065 0.065"/>
+        <parent link="segment7"/>
+        <child link="vacuum_gripper_down"/>
+        <axis xyz="0 1 1"/>
+        <limit effort="30.0" lower="-0.01" upper="0.035" velocity="0.1"/>
+        <mimic joint="vacuum_up_joint"/>
+    </joint>
 </robot>

Commit message: relax the joint limits of joint 0 a little more, moveit complains about violation => probably floating point issue

File: src/cobot_model/urdf/robot_model.urdf.xacro (robot description, xacro)
@@ -408,5 +408,5 @@
         <child link="lin_axis_carriage" />
         <axis xyz="0 0 1" />
-        <limit effort="300.0" velocity="3.141593" lower="-0.0001" upper="0.894" />
+        <limit effort="300.0" velocity="3.141593" lower="-0.001" upper="0.894" />
     </joint>
     <joint name="mount_fixture" type="fixed">

Commit message: update finger gripper position and state

File: src/cobot_model/urdf/robot_model.urdf.xacro (robot description, xacro)
@@ -474,16 +474,16 @@
     </joint>
     <joint name="finger1_joint" type="prismatic">
-        <origin rpy="0.0 0.0 0.0" xyz="0.0 -0.065 0.065"/>
+        <origin rpy="0.0 0.0 0.0" xyz="-0.04 -0.065 0.065"/>
         <parent link="segment7" />
         <child link="finger1" />
-        <axis xyz="-1 0 0" />
-        <limit effort="30.0" velocity="0.1" lower="-0.01" upper="0.015" />
+        <axis xyz="1 0 0" />
+        <limit effort="30.0" velocity="0.1" lower="-0.01" upper="0.041" />
     </joint>
     <joint name="finger2_joint" type="prismatic">
-        <origin rpy="0.0 0.0 0.0" xyz="0.0 -0.065 0.065"/>
+        <origin rpy="0.0 0.0 0.0" xyz="0.04 -0.065 0.065"/>
         <parent link="segment7" />
         <child link="finger2" />
-        <axis xyz="1 0 0" />
-        <limit effort="30.0" velocity="0.1" lower="-0.01" upper="0.015" />
+        <axis xyz="-1 0 0" />
+        <limit effort="30.0" velocity="0.1" lower="-0.01" upper="0.041" />
         <mimic joint="finger1_joint" />
     </joint>
@@ -493,5 +493,5 @@
         <child link="vacuum_gripper_up"/>
         <axis xyz="0 1 1"/>
-        <limit effort="30.0" lower="-0.01" upper="0.035" velocity="0.1"/>
+        <limit effort="30.0" lower="-0.01" upper="0.036" velocity="0.1"/>
     </joint>
     <joint name="vacuum_down_joint" type="prismatic">
@@ -500,5 +500,5 @@
         <child link="vacuum_gripper_down"/>
         <axis xyz="0 1 1"/>
-        <limit effort="30.0" lower="-0.01" upper="0.035" velocity="0.1"/>
+        <limit effort="30.0" lower="-0.01" upper="0.036" velocity="0.1"/>
         <mimic joint="vacuum_up_joint"/>
     </joint>

Commit message: adjust positions for finger gripper

File: src/cobot_model/urdf/robot_model.urdf.xacro (robot description, xacro)
@@ -474,16 +474,16 @@
     </joint>
     <joint name="finger1_joint" type="prismatic">
-        <origin rpy="0.0 0.0 0.0" xyz="-0.04 -0.065 0.065"/>
+        <origin rpy="0.0 0.0 0.0" xyz="-0.02 -0.065 0.065"/>
         <parent link="segment7" />
         <child link="finger1" />
         <axis xyz="1 0 0" />
-        <limit effort="30.0" velocity="0.1" lower="-0.01" upper="0.041" />
+        <limit effort="30.0" velocity="0.1" lower="-0.01" upper="0.029" />
     </joint>
     <joint name="finger2_joint" type="prismatic">
-        <origin rpy="0.0 0.0 0.0" xyz="0.04 -0.065 0.065"/>
+        <origin rpy="0.0 0.0 0.0" xyz="0.02 -0.065 0.065"/>
         <parent link="segment7" />
         <child link="finger2" />
         <axis xyz="-1 0 0" />
-        <limit effort="30.0" velocity="0.1" lower="-0.01" upper="0.041" />
+        <limit effort="30.0" velocity="0.1" lower="-0.01" upper="0.029" />
         <mimic joint="finger1_joint" />
     </joint>
@@ -492,4 +492,6 @@
         <parent link="segment7"/>
         <child link="vacuum_gripper_up"/>
+        <!-- The head of the cobot is rotated by 45deg => joint moves in two directions -->
+        <!-- TODO @rharbach normalize: <axis xyz="0 0.70710678 0.70710678"/> -->
         <axis xyz="0 1 1"/>
         <limit effort="30.0" lower="-0.01" upper="0.036" velocity="0.1"/>

Commit message: remove obsolete comment

File: src/cobot_model/urdf/robot_model.urdf.xacro (robot description, xacro)
@@ -493,5 +493,4 @@
         <child link="vacuum_gripper_up"/>
         <!-- The head of the cobot is rotated by 45deg => joint moves in two directions -->
-        <!-- TODO @rharbach normalize: <axis xyz="0 0.70710678 0.70710678"/> -->
         <axis xyz="0 1 1"/>
         <limit effort="30.0" lower="-0.01" upper="0.036" velocity="0.1"/>
