Commit message: follow right hand rule + simplify rotations + add additional tcps

File: src/cobot_model/urdf/robot_model.urdf.xacro (robot description, xacro)
@@ -15,15 +15,15 @@
             <origin rpy="0.0 0.0 0.0" xyz="0.0 0.0 0.0" />
             <geometry>
-                <mesh filename="package://cobot_model/meshes/visual/axis_visual.dae" scale="0.001 0.001 0.001" />
-                <material name="silver">
-                    <color rgba="1.0 1.0 1.0 1.0" />
-                </material>
-            </geometry>
-        </visual>
-        <collision>
-            <xacro:if value="${'$(arg use_collision_meshes)' == 'true'}">
-                <origin rpy="0.0 0.0 0.0" xyz="0.0 0.0 0.0" />
-                <geometry>
-                    <mesh filename="package://cobot_model/meshes/collision/axis_collision.dae" scale="0.001 0.001 0.001" />
+                <mesh filename="package://cobot_model/meshes/visual/axis_visual.stl"/>
+            </geometry>
+            <material name="axis_material">
+                <color rgba="0.58 0.58 0.58 1.0"/>
+            </material>
+        </visual>
+        <collision>
+            <xacro:if value="${'$(arg use_collision_meshes)' == 'true'}">
+                <origin rpy="0.0 0.0 0.0" xyz="0.0 0.0 0.0" />
+                <geometry>
+                   <mesh filename="package://cobot_model/meshes/collision/axis_collision.stl"/>
                 </geometry>
             </xacro:if>
@@ -45,15 +45,15 @@
              <origin rpy="0.0 0.0 0.0" xyz="0.0 0.0 0.0" />
             <geometry>
-                <mesh filename="package://cobot_model/meshes/visual/carriage_real_visual.dae" scale="0.001 0.001 0.001" />
-                <material name="silver">
-                    <color rgba="1.0 1.0 1.0 1.0" />
-                </material>
-            </geometry>
-        </visual>
-        <collision>
-            <xacro:if value="${'$(arg use_collision_meshes)' == 'true'}">
-                <origin rpy="0.0 0.0 0.0" xyz="0.0 0.0 0.0" />
-                <geometry>
-                   <mesh filename="package://cobot_model/meshes/visual/carriage_real_visual.dae" scale="0.001 0.001 0.001" />
+               <mesh filename="package://cobot_model/meshes/visual/carriage_visual.stl"/>
+            </geometry>
+            <material name="axis_material">
+                <color rgba="0.58 0.58 0.58 1.0"/>
+            </material>
+        </visual>
+        <collision>
+            <xacro:if value="${'$(arg use_collision_meshes)' == 'true'}">
+                <origin rpy="0.0 0.0 0.0" xyz="0.0 0.0 0.0" />
+                <geometry>
+                    <mesh filename="package://cobot_model/meshes/collision/carriage_collision.stl"/>
                 </geometry>
             </xacro:if>
@@ -75,5 +75,6 @@
              <origin rpy="0.0 0.0 0.0" xyz="0.0 0.0 0.0" />
             <geometry>
-                <mesh filename="package://cobot_model/meshes/visual/segment_01_logo.dae" scale="0.001 0.001 0.001" />
+                <!-- using a DAE mesh to display logos -->
+               <mesh filename="package://cobot_model/meshes/visual/segment_01_logo.dae"/>
             </geometry>
             <material name="segment1_material">
@@ -85,5 +86,5 @@
                 <origin rpy="0.0 0.0 0.0" xyz="0.0 0.0 0.0" />
                 <geometry>
-                    <mesh filename="package://cobot_model/meshes/collision/segment01_collision.stl" scale="0.001 0.001 0.001" />
+                    <mesh filename="package://cobot_model/meshes/collision/segment01_collision.stl"/>
                 </geometry>
             </xacro:if>
@@ -105,5 +106,5 @@
             <origin rpy="0.0 0.0 0.0" xyz="0.0 0.0 0.0" />
             <geometry>
-                <mesh filename="package://cobot_model/meshes/visual/segment02_visual.stl" scale="0.001 0.001 0.001" />
+                <mesh filename="package://cobot_model/meshes/visual/segment02_visual.stl"/>
             </geometry>
             <material name="segment2_material">
@@ -115,5 +116,5 @@
                 <origin rpy="0.0 0.0 0.0" xyz="0.0 0.0 0.0" />
                 <geometry>
-                    <mesh filename="package://cobot_model/meshes/collision/segment02_collision.stl" scale="0.001 0.001 0.001" />
+                   <mesh filename="package://cobot_model/meshes/collision/segment02_collision.stl"/>
                 </geometry>
             </xacro:if>
@@ -135,5 +136,5 @@
             <origin rpy="0.0 0.0 0.0" xyz="0.0 0.0 0.0" />
             <geometry>
-                <mesh filename="package://cobot_model/meshes/visual/segment03_visual.stl" scale="0.001 0.001 0.001" />
+                <mesh filename="package://cobot_model/meshes/visual/segment03_visual.stl"/>
             </geometry>
             <material name="segment3_material">
@@ -145,5 +146,5 @@
                 <origin rpy="0.0 0.0 0.0" xyz="0.0 0.0 0.0" />
                 <geometry>
-                    <mesh filename="package://cobot_model/meshes/collision/segment03_collision.stl" scale="0.001 0.001 0.001" />
+                    <mesh filename="package://cobot_model/meshes/collision/segment03_collision.stl"/>
                 </geometry>
             </xacro:if>
@@ -165,5 +166,5 @@
             <origin rpy="0.0 0.0 0.0" xyz="0.0 0.0 0.0" />
             <geometry>
-                <mesh filename="package://cobot_model/meshes/visual/segment04_visual.stl" scale="0.001 0.001 0.001" />
+                <mesh filename="package://cobot_model/meshes/visual/segment04_visual.stl"/>
             </geometry>
             <material name="segment4_material">
@@ -175,5 +176,5 @@
                 <origin rpy="0.0 0.0 0.0" xyz="0.0 0.0 0.0" />
                 <geometry>
-                    <mesh filename="package://cobot_model/meshes/collision/segment04_collision.stl" scale="0.001 0.001 0.001" />
+                    <mesh filename="package://cobot_model/meshes/collision/segment04_collision.stl"/>
                 </geometry>
             </xacro:if>
@@ -195,5 +196,5 @@
             <origin rpy="0.0 0.0 0.0" xyz="0.0 0.0 0.0" />
             <geometry>
-                <mesh filename="package://cobot_model/meshes/visual/segment05_power_visual.stl" scale="0.001 0.001 0.001" />
+                <mesh filename="package://cobot_model/meshes/visual/segment05_visual.stl"/>
             </geometry>
             <material name="segment5_material">
@@ -205,5 +206,5 @@
                 <origin rpy="0.0 0.0 0.0" xyz="0.0 0.0 0.0" />
                 <geometry>
-                    <mesh filename="package://cobot_model/meshes/collision/segment05_power_collision.stl" scale="0.001 0.001 0.001" />
+                    <mesh filename="package://cobot_model/meshes/collision/segment05_collision.stl"/>
                 </geometry>
             </xacro:if>
@@ -225,5 +226,5 @@
             <origin rpy="0.0 0.0 0.0" xyz="0.0 0.0 0.0" />
             <geometry>
-                <mesh filename="package://cobot_model/meshes/visual/segment06_power_visual.stl" scale="0.001 0.001 0.001" />
+                <mesh filename="package://cobot_model/meshes/visual/segment06_visual.stl"/>
             </geometry>
             <material name="segment6_material">
@@ -235,5 +236,5 @@
                 <origin rpy="0.0 0.0 0.0" xyz="0.0 0.0 0.0" />
                 <geometry>
-                    <mesh filename="package://cobot_model/meshes/collision/segment06_power_collision.stl" scale="0.001 0.001 0.001" />
+                    <mesh filename="package://cobot_model/meshes/collision/segment06_collision.stl"/>
                 </geometry>
              </xacro:if>
@@ -258,5 +259,5 @@
             </material>
             <geometry>
-                <mesh filename="package://cobot_model/meshes/visual/segment07_real_visual.stl" scale="0.001 0.001 0.001"/>
+                 <mesh filename="package://cobot_model/meshes/visual/segment07_visual.stl" />
             </geometry>
         </visual>
@@ -265,5 +266,5 @@
                 <origin rpy="0.0 0.0 0.0" xyz="0.0 0.0 0.0"/>
                 <geometry>
-                    <mesh filename="package://cobot_model/meshes/collision/segment07_real_collision.stl" scale="0.001 0.001 0.001"/>
+                    <mesh filename="package://cobot_model/meshes/collision/segment07_collision.stl"/>
                 </geometry>
             </xacro:if>
@@ -280,21 +281,20 @@
            <inertia ixx="0.02693367" iyy="0.01533367" izz="0.02185067" ixy="0.0" ixz="0.0" iyz="0.0" />
         </inertial>
-  </link>
-    <link name="TCP"/>
+    </link>
     <link name="finger1">
         <visual>
-           <origin rpy="0.0 0.0 0.0" xyz="0.0 0.065 -0.065"/>
+            <origin rpy="0.0 0.0 0.0" xyz="0.0 0.0 0.0"/>
             <material name="silver">
                 <color rgba="0.629 0.629 0.625 1.0" />
             </material>
             <geometry>
-                <mesh filename="package://cobot_model/meshes/visual/finger01_real_visual.stl" scale="0.001 0.001 0.001" />
-            </geometry>
-        </visual>
-        <collision>
-            <xacro:if value="${'$(arg use_collision_meshes)' == 'true'}">
-                <origin rpy="0.0 0.0 0.0" xyz="0.0 0.065 -0.065"/>
-                <geometry>
-                    <mesh filename="package://cobot_model/meshes/collision/finger01_real_collision.stl" scale="0.001 0.001 0.001" />
+                <mesh filename="package://cobot_model/meshes/visual/finger01_visual.stl"/>
+            </geometry>
+        </visual>
+        <collision>
+            <xacro:if value="${'$(arg use_collision_meshes)' == 'true'}">
+                <origin rpy="0.0 0.0 0.0" xyz="0.0 0.0 0.0"/>
+                <geometry>
+                        <mesh filename="package://cobot_model/meshes/collision/finger01_collision.stl"/>
                 </geometry>
             </xacro:if>
@@ -314,17 +314,17 @@
     <link name="finger2">
         <visual>
-            <origin rpy="0.0 0.0 0.0" xyz="0.0 0.065 -0.065"/>
+            <origin rpy="0.0 0.0 0.0" xyz="0.0 0.0 0.0"/>
             <material name="silver">
                 <color rgba="0.629 0.629 0.625 1.0" />
             </material>
             <geometry>
-                <mesh filename="package://cobot_model/meshes/visual/finger02_real_visual.stl" scale="0.001 0.001 0.001" />
-            </geometry>
-        </visual>
-        <collision>
-            <xacro:if value="${'$(arg use_collision_meshes)' == 'true'}">
-                <origin rpy="0.0 0.0 0.0" xyz="0.0 0.065 -0.065"/>
-                <geometry>
-                    <mesh filename="package://cobot_model/meshes/collision/finger02_real_collision.stl" scale="0.001 0.001 0.001" />
+                <mesh filename="package://cobot_model/meshes/visual/finger02_visual.stl"/>
+            </geometry>
+        </visual>
+        <collision>
+            <xacro:if value="${'$(arg use_collision_meshes)' == 'true'}">
+                <origin rpy="0.0 0.0 0.0" xyz="0.0 0.0 0.0"/>
+                <geometry>
+                    <mesh filename="package://cobot_model/meshes/collision/finger02_collision.stl"/>
                 </geometry>
             </xacro:if>
@@ -344,17 +344,17 @@
     <link name="vacuum_gripper_up">
     <visual>
-      <origin rpy="0.0 0.0 0.0" xyz="0.0 0.026 -0.103"/>
+      <origin rpy="0.0 0.0 0.0" xyz="0.0 0.0 0.0"/>
       <material name="silver">
         <color rgba="0.629 0.629 0.625 1.0"/>
       </material>
       <geometry>
-        <mesh filename="package://cobot_model/meshes/visual/vacuum_gripper_up_visual.stl" scale="0.001 0.001 0.001"/>
+        <mesh filename="package://cobot_model/meshes/visual/vacuum_visual.stl"/>
       </geometry>
     </visual>
     <collision>
     <xacro:if value="${'$(arg use_collision_meshes)' == 'true'}">
-        <origin rpy="0.0 0.0 0.0" xyz="0.0 0.026 -0.103"/>
+        <origin rpy="0.0 0.0 0.0" xyz="0.0 0.0 0.0"/>
         <geometry>
-            <mesh filename="package://cobot_model/meshes/collision/vacuum_gripper_up_collision.stl" scale="0.001 0.001 0.001"/>
+            <mesh filename="package://cobot_model/meshes/collision/vacuum_collision.stl"/>
         </geometry>
     </xacro:if>
@@ -374,17 +374,19 @@
   <link name="vacuum_gripper_down">
     <visual>
-      <origin rpy="0.0 0.0 0.0" xyz="0.0 0.026 -0.103"/>
+      <origin rpy="0.0 0.0 0.0" xyz="0.0 0.0 0.0"/>
       <material name="silver">
         <color rgba="0.629 0.629 0.625 1.0"/>
       </material>
       <geometry>
-        <mesh filename="package://cobot_model/meshes/visual/vacuum_gripper_down_visual.stl" scale="0.001 0.001 0.001"/>
+        <!-- using the same mesh as for the upper vacuum gripper (they look the same in the model) -->
+        <mesh filename="package://cobot_model/meshes/visual/vacuum_visual.stl"/>
       </geometry>
     </visual>
     <collision>
         <xacro:if value="${'$(arg use_collision_meshes)' == 'true'}">
-            <origin rpy="0.0 0.0 0.0" xyz="0.0 0.026 -0.103"/>
-            <geometry>
-                <mesh filename="package://cobot_model/meshes/collision/vacuum_gripper_down_collision.stl" scale="0.001 0.001 0.001"/>
+            <origin rpy="0.0 0.0 0.0" xyz="0.0 0.0 0.0"/>
+            <geometry>
+                <!-- using the same mesh as for the upper vacuum gripper (they look the same in the model) -->
+                <mesh filename="package://cobot_model/meshes/collision/vacuum_collision.stl"/>
             </geometry>
         </xacro:if>
@@ -402,4 +404,17 @@
     </inertial>
   </link>
+    <!-- the virtual links (defined for readbility)
+    We follow the following structure:
+    link_0 -> ... -> link_n -> flange -> tool_base
+                                            -> gripper_tcp
+                                            -> vacuump_up_tcp
+                                            -> vacuum_down_tcp
+    This enables independent tool center points (one per tool)
+    -->
+    <link name="flange"/>
+    <link name="tool_base"/>
+    <link name="gripper_tcp"/>
+    <link name="vacuum_up_tcp"/>
+    <link name="vacuum_down_tcp"/>
     <!-- Joints -->
     <joint name="joint_0" type="prismatic">
@@ -411,10 +426,10 @@
     </joint>
     <joint name="mount_fixture" type="fixed">
-        <origin rpy="0.0 0.0 0.0" xyz="0.0 0.37 0.52" />
+        <origin rpy="0.0 0.0 0.0" xyz="0.0 -0.37 0.52" />
         <parent link="lin_axis_carriage" />
         <child link="segment1" />
     </joint>
     <joint name="joint_1" type="revolute">
-        <origin rpy="0.0 0.0 -3.14" xyz="0.0 0.0 0.0" />
+        <origin rpy="0.0 0.0 0.0" xyz="0.0 0.0 0.0"/>
         <parent link="segment1" />
         <child link="segment2" />
@@ -424,5 +439,5 @@
     </joint>
     <joint name="joint_2" type="revolute">
-        <origin rpy="1.5708 -1.5708 0.0" xyz="0.0 -0.111 0.118" />
+         <origin rpy="1.57 0.0 0.0" xyz="0.0 -0.111 0.118"/>
         <parent link="segment2" />
         <child link="segment3" />
@@ -432,5 +447,5 @@
     </joint>
     <joint name="joint_3" type="revolute">
-        <origin rpy="0.0 0.0 -1.57" xyz="0.254 0.0 0.06" />
+         <origin rpy="0.0 0.0 0.0" xyz="0.0 0.254 0.06"/>
         <parent link="segment3" />
         <child link="segment4" />
@@ -440,5 +455,5 @@
     </joint>
     <joint name="joint_4" type="revolute">
-        <origin rpy="-1.5708 0.0 -1.5708" xyz="0.062 0.0 -0.168"/>
+        <origin rpy="0.0 1.570 0.0" xyz="0.062 0.0 -0.168"/>
         <parent link="segment4" />
         <child link="segment5" />
@@ -448,5 +463,5 @@
     </joint>
     <joint name="joint_5" type="revolute">
-        <origin rpy="-1.570 -1.570 0.0" xyz="0.0 0.042 0.183" />
+        <origin rpy="0.0 1.57 0.0" xyz="0.042 0.0 0.183"/>
         <parent link="segment5" />
         <child link="segment6" />
@@ -456,5 +471,5 @@
     </joint>
     <joint name="joint_6" type="revolute">
-        <origin rpy="0.0 1.57 0.0" xyz="0.156 0.0 -0.04"/>
+        <origin rpy="0.0 -1.570 0.0" xyz="-0.156 0.0 -0.04"/>
         <parent link="segment6"/>
         <child link="segment7"/>
@@ -463,9 +478,4 @@
         <dynamics damping="0.0" friction="0.0"/>
     </joint>
-    <joint name="JFix_TCP" type="fixed">
-        <origin rpy="-0.785 0.0 0.0" xyz="0.0 -0.02 0.12"/>
-        <parent link="segment7"/>
-        <child link="TCP"/>
-    </joint>
    <joint name="JFix_Base" type="fixed">
         <origin rpy="0.0 0.0 0.0" xyz="0.0 0.0 0.0" />
@@ -473,33 +483,61 @@
         <child link="lin_axis" />
     </joint>
+    <joint name="flange_fixed" type="fixed">
+        <origin rpy="0.0 0.0 0.0" xyz="0.0 0.0 0.0"/>
+        <parent link="segment7"/>
+        <child link="flange"/>
+     </joint>
+    <joint name="tool_mount" type="fixed">
+        <!-- tilt tool base by 45 deg + move coordinate frame -->
+        <origin rpy="0.785 0.0 0.0" xyz="0.0 0.072 0.060"/>
+        <parent link="flange"/>
+        <child link="tool_base"/>
+    </joint>
+    <joint name="tool_base_gripper_tcp" type="fixed">
+        <!-- place gripper TCP in between the fingers (z-direction) -->
+        <origin rpy="0.0 0.0 0.0" xyz="0.0 0.0 0.075"/>
+        <parent link="tool_base"/>
+        <child link="gripper_tcp"/>
+    </joint>
     <joint name="finger1_joint" type="prismatic">
-        <origin rpy="0.0 0.0 0.0" xyz="-0.02 -0.065 0.065"/>
-        <parent link="segment7" />
+        <origin rpy="0.0 0.0 0.0" xyz="0.0 0.0 0.0"/>
+        <parent link="tool_base" />
         <child link="finger1" />
+        <axis xyz="-1 0 0" />
+        <limit effort="30.0" velocity="0.1" lower="-0.01" upper="0.029" />
+    </joint>
+    <joint name="finger2_joint" type="prismatic">
+        <origin rpy="0.0 0.0 0.0" xyz="0.0 0.0 0.0"/>
+        <parent link="tool_base" />
+        <child link="finger2" />
         <axis xyz="1 0 0" />
         <limit effort="30.0" velocity="0.1" lower="-0.01" upper="0.029" />
-    </joint>
-    <joint name="finger2_joint" type="prismatic">
-        <origin rpy="0.0 0.0 0.0" xyz="0.02 -0.065 0.065"/>
-        <parent link="segment7" />
-        <child link="finger2" />
-        <axis xyz="-1 0 0" />
-        <limit effort="30.0" velocity="0.1" lower="-0.01" upper="0.029" />
         <mimic joint="finger1_joint" />
     </joint>
     <joint name="vacuum_up_joint" type="prismatic">
-        <origin rpy="0.0 0.0 0.0" xyz="0.0 -0.065 0.065"/>
-        <parent link="segment7"/>
+        <origin rpy="0.0 0.0 0.0" xyz="0.0 0.035 0.0"/>
+        <parent link="tool_base"/>
         <child link="vacuum_gripper_up"/>
-        <!-- The head of the cobot is rotated by 45deg => joint moves in two directions -->
-        <axis xyz="0 1 1"/>
+        <axis xyz="0 0 1"/>
         <limit effort="30.0" lower="-0.01" upper="0.036" velocity="0.1"/>
     </joint>
+    <joint name="vacuum_up_to_tcp" type="fixed">
+        <!-- place TCP at the end of the tool (z-direction) -->
+        <origin rpy="0.0 0.0 0.0" xyz="0.0 0.0 0.07"/>
+        <parent link="vacuum_gripper_up"/>
+        <child link="vacuum_up_tcp"/>
+    </joint>
     <joint name="vacuum_down_joint" type="prismatic">
-        <origin rpy="0.0 0.0 0.0" xyz="0.0 -0.065 0.065"/>
-        <parent link="segment7"/>
+        <origin rpy="0.0 0.0 0.0" xyz="0.0 -0.035 0.0"/>
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
Commit message: modify simple geometric collisions to match robot model

File: src/cobot_model/urdf/robot_model.urdf.xacro (robot description, xacro)
@@ -29,5 +29,5 @@
             </xacro:if>
             <xacro:unless value="${'$(arg use_collision_meshes)' == 'true'}">
-                <origin rpy="0.0 0.0 0.0" xyz="0.0 0.03 0.6"/>
+                <origin rpy="0.0 0.0 0.0" xyz="0.0 -0.03 0.6"/>
                 <geometry>
                     <box size="0.162 0.069 1.21"/>
@@ -59,5 +59,5 @@
             </xacro:if>
             <xacro:unless value="${'$(arg use_collision_meshes)' == 'true'}">
-                <origin rpy="0.0 0.0 0.0" xyz="0.06 0.26 0.2"/>
+                <origin rpy="0.0 0.0 0.0" xyz="-0.06 -0.26 0.2"/>
                 <geometry>
                     <box size="0.302 0.431 0.02"/>
@@ -150,5 +150,5 @@
             </xacro:if>
             <xacro:unless value="${'$(arg use_collision_meshes)' == 'true'}">
-                <origin rpy="0.0 1.57 0.0" xyz="0.126 0.0 0.06"/>
+                <origin rpy="1.57 0.0 0.0" xyz="0.0 0.126 0.06"/>
                 <geometry>
                     <cylinder radius="0.06" length="0.372"/>
@@ -240,5 +240,5 @@
              </xacro:if>
             <xacro:unless value="${'$(arg use_collision_meshes)' == 'true'}">
-                <origin rpy="0.0 1.57 0.0" xyz="0.12 0.0 -0.04"/>
+                <origin rpy="0.0 1.57 0.0" xyz="-0.12 0.0 -0.04"/>
                 <geometry>
                     <cylinder length="0.15" radius="0.04"/>
@@ -270,5 +270,5 @@
             </xacro:if>
             <xacro:unless value="${'$(arg use_collision_meshes)' == 'true'}">
-                <origin rpy="-0.786 0.0 0.0" xyz="0.0 -0.1 0.05"/>
+                <origin rpy="-0.786 0.0 0.0" xyz="0.0 0.1 0.05"/>
                 <geometry>
                     <box size="0.124 0.135 0.14"/>
@@ -300,5 +300,5 @@
             </xacro:if>
             <xacro:unless value="${'$(arg use_collision_meshes)' == 'true'}">
-                <origin rpy="-0.786 0.25 0.0" xyz="-0.020 0.040 0.036"/>
+                <origin rpy="0.0 -0.25 0.0" xyz="0.046 0.0 0.056"/>
                 <geometry>
                     <cylinder length="0.10" radius="0.01"/>
@@ -330,5 +330,5 @@
             </xacro:if>
             <xacro:unless value="${'$(arg use_collision_meshes)' == 'true'}">
-                <origin rpy="-0.786 -0.25 0.0" xyz="0.020 0.040 0.036"/>
+                <origin rpy="0.0 0.25 0.0" xyz="-0.046 0.0 0.056"/>
                 <geometry>
                     <cylinder length="0.10" radius="0.01"/>
@@ -360,5 +360,5 @@
     </xacro:if>
     <xacro:unless value="${'$(arg use_collision_meshes)' == 'true'}">
-        <origin rpy="-0.786 0.0 0.0" xyz="0.0 -0.008 0.042"/>
+        <origin rpy="0.0 0.0 0.0" xyz="0.0 0.0 0.03"/>
         <geometry>
             <cylinder length="0.10" radius="0.01"/>
@@ -392,5 +392,5 @@
         </xacro:if>
        <xacro:unless value="${'$(arg use_collision_meshes)' == 'true'}">
-            <origin rpy="-0.786 0.0 0.0" xyz="0.0 0.042 -0.008"/>
+            <origin rpy="0.0 0.0 0.0" xyz="0.0 0.0 0.03"/>
             <geometry>
                 <cylinder length="0.10" radius="0.01"/>
