Commit message: update inertia values to match updated rotations in model

File: src/cobot_model/urdf/robot_model.urdf.xacro (robot description, xacro)
@@ -37,5 +37,5 @@
         <inertial>
             <mass value="8.6" />
-            <origin rpy="0.0 0.0 0.0" xyz="0.0 0.0 0.6" />
+            <origin rpy="0.0 0.0 0.0" xyz="0.0 -0.03 0.6" />
             <inertia ixx="1.03466672" iyy="1.0433778" izz="0.01404452" ixy="0.0" ixz="0.0" iyz="0.0" />
         </inertial>
@@ -67,5 +67,5 @@
         <inertial>
             <mass value="0.7" />
-            <origin rpy="0.0 0.0 0.0" xyz="0.0 0.0 0.11" />
+            <origin rpy="0.0 0.0 0.0" xyz="0.0 -0.03 0.11" />
             <inertia ixx="0.00287479" iyy="0.00415339" izz="0.00138151" ixy="0.0" ixz="0.0" iyz="0.0" />
         </inertial>
@@ -158,6 +158,6 @@
         <inertial>
             <mass value="2.5" />
-            <origin rpy="0.0 0.0 0.0" xyz="0.126 0.0 0.06" />
-            <inertia ixx="0.01325083" ixy="0.0" ixz="-0.0189" iyy="0.06515833" iyz="0.0" izz="0.05607417" />
+            <origin rpy="0.0 0.0 0.0" xyz="0.0 0.126 0.06" />
+            <inertia ixx="0.06515833" ixy="0.0" ixz="0.0" iyy="0.01316667" iyz="-0.0189" izz="0.05607417" />
         </inertial>
     </link>
@@ -217,7 +217,7 @@
         </collision>
         <inertial>
-            <mass value="1.1" />
+            <mass value="3.0" />
             <origin rpy="0.0 0.0 0.0" xyz="0.0 0.0 0.071" />
-            <inertia ixx="0.00623544" iyy="0.00623544" izz="0.00277255" ixy="0.0" ixz="0.0" iyz="0.0" />
+            <inertia ixx="0.02173675" iyy="0.02173675" izz="0.0075615" ixy="0.0" ixz="0.0" iyz="0.0" />
         </inertial>
     </link>
@@ -248,5 +248,5 @@
         <inertial>
             <mass value="1.5" />
-            <origin rpy="0.0 0.0 0.0" xyz="0.05 0.0 0.0" />
+            <origin rpy="0.0 0.0 0.0" xyz="-0.05 0.0 0.0" />
             <inertia ixx="0.00319363" iyy="0.00513113" izz="0.0061625" ixy="0.0" ixz="0.0" iyz="0.0" />
         </inertial>
@@ -278,6 +278,8 @@
         <inertial>
             <mass value="4.0"/>
-            <origin rpy="0.0 0.0 0.0" xyz="0.0 -0.09 0.04"/>
-           <inertia ixx="0.02693367" iyy="0.01533367" izz="0.02185067" ixy="0.0" ixz="0.0" iyz="0.0" />
+            <!-- tilt the inertia tensor by 45 deg to match the actual mesh
+                 => same tilt is applied in the tool_base link -->
+            <origin rpy="0.785 0.0 0.0" xyz="0.0 0.09 0.04"/>
+           <inertia ixx="0.01533367" iyy="0.02185067" izz="0.02693367" ixy="0.0" ixz="0.0" iyz="0.0" />
         </inertial>
     </link>
@@ -308,5 +310,7 @@
         <inertial>
             <mass value="0.05" />
-            <origin rpy="-0.785 0.0 0.0" xyz="0.02 0.03 0.03" />
+            <!-- <origin rpy="-0.785 0.0 0.0" xyz="0.02 0.03 0.03" / -->
+            <origin rpy="0.0 -0.25 0.0" xyz="0.046 0.0 0.056"/>
+            <!-- <origin rpy="0.0 0.0 0.0" xyz="0.0 0.0 0.0" /> -->
             <inertia ixx="3.46666667e-05" iyy="2.64166667e-05" izz="1.78833333e-05" ixy="0.0" ixz="0.0" iyz="0.0" />
         </inertial>
@@ -338,5 +342,5 @@
         <inertial>
             <mass value="0.05" />
-            <origin rpy="-0.785 0.0 0.0" xyz="-0.02 0.03 0.03" />
+            <origin rpy="0.0 0.25 0.0" xyz="-0.046 0.0 0.056"/>
             <inertia ixx="3.46666667e-05" iyy="2.64166667e-05" izz="1.78833333e-05" ixy="0.0" ixz="0.0" iyz="0.0" />
         </inertial>
@@ -368,6 +372,6 @@
     <inertial>
       <mass value="0.05"/>
-      <origin rpy="-0.785 0.0 0.0" xyz="0.0 0.001 0.052"/>
-      <inertia ixx="3.46666667e-05" ixy="0.0" ixz="0.0" iyy="2.64166667e-05" iyz="0.0" izz="1.78833333e-05"/>
+      <origin rpy="0.0 0.0 0.0" xyz="0.0 0.0 0.05"/>
+      <inertia ixx="2.08333333e-05" ixy="0.0" ixz="0.0" iyy="2.08333333e-05" iyz="0.0" izz="2.08333333e-05"/>
     </inertial>
   </link>
@@ -400,6 +404,6 @@
     <inertial>
       <mass value="0.05"/>
-      <origin rpy="-0.785 0.0 0.0" xyz="0.0 0.052 0.001"/>
-      <inertia ixx="3.46666667e-05" ixy="0.0" ixz="0.0" iyy="2.64166667e-05" iyz="0.0" izz="1.78833333e-05"/>
+      <origin rpy="0.0 0.0 0.0" xyz="0.0 0.0 0.05"/>
+      <inertia ixx="2.08333333e-05" ixy="0.0" ixz="0.0" iyy="2.08333333e-05" iyz="0.0" izz="2.08333333e-05"/>
     </inertial>
   </link>

Commit message: add custom tcp frames to model

File: src/cobot_model/urdf/robot_model.urdf.xacro (robot description, xacro)
@@ -408,17 +408,35 @@
     </inertial>
   </link>
-    <!-- the virtual links (defined for readbility)
-    We follow the following structure:
+    <!-- the virtual links
+    We follow the following structure to enable individual TCPs per tool:
     link_0 -> ... -> link_n -> flange -> tool_base
                                             -> gripper_tcp
+                                                -> gripper_tcp_world
+                                                    -> gripper_tcp_world_tilted_up
+                                                    -> gripper_tcp_world_tilted_down
                                             -> vacuump_up_tcp
                                             -> vacuum_down_tcp
-    This enables independent tool center points (one per tool)
+    The additional TCP frames are defined to ease up IK requests (omitting transformations in code):
+        * TCP in world frame: all rotations inverted
+            => cobot can move to any point in its neutral orientation
+        * TCP in world tilted z up: compensates the natural tilt in the physical model, Z+ is up
+            => cobot will approach any object with a neutral orientation from above
+        * TCP in world tilted z down: same as previous but Z+ pointing down
+            => cobot will approach objects from above that have an inverted orientation
     -->
     <link name="flange"/>
     <link name="tool_base"/>
     <link name="gripper_tcp"/>
+    <link name="gripper_tcp_world"/>
+    <link name="gripper_tcp_world_tilted_up"/>
+    <link name="gripper_tcp_world_tilted_down"/>
     <link name="vacuum_up_tcp"/>
+    <link name="vacuum_up_tcp_world"/>
+    <link name="vacuum_up_tcp_world_tilted_up"/>
+    <link name="vacuum_up_tcp_world_tilted_down"/>
     <link name="vacuum_down_tcp"/>
+    <link name="vacuum_down_tcp_world"/>
+    <link name="vacuum_down_tcp_world_tilted_up"/>
+    <link name="vacuum_down_tcp_world_tilted_down"/>
     <!-- Joints -->
     <joint name="joint_0" type="prismatic">
@@ -443,5 +461,5 @@
     </joint>
     <joint name="joint_2" type="revolute">
-         <origin rpy="1.57 0.0 0.0" xyz="0.0 -0.111 0.118"/>
+        <origin rpy="1.57 0.0 0.0" xyz="0.0 -0.111 0.118"/>
         <parent link="segment2" />
         <child link="segment3" />
@@ -498,9 +516,27 @@
         <child link="tool_base"/>
     </joint>
-    <joint name="tool_base_gripper_tcp" type="fixed">
+    <joint name="gripper_tcp_mount" type="fixed">
         <!-- place gripper TCP in between the fingers (z-direction) -->
         <origin rpy="0.0 0.0 0.0" xyz="0.0 0.0 0.075"/>
         <parent link="tool_base"/>
         <child link="gripper_tcp"/>
+    </joint>
+    <joint name="gripper_tcp_world_mount" type="fixed">
+        <!-- reverse all previous rotations -->
+        <origin rpy="-3.14 -0.785 1.57" xyz="0.0 0.0 0.0"/>
+        <parent link="gripper_tcp"/>
+        <child link="gripper_tcp_world"/>
+    </joint>
+    <joint name="gripper_tcp_world_tilted_up_mount" type="fixed">
+        <!-- tilt gripper tcp in world frame by -45 deg to compensate for natural tilt -->
+        <origin rpy="0.0 -0.785 0.0" xyz="0.0 0.0 0.0"/>
+        <parent link="gripper_tcp_world"/>
+        <child link="gripper_tcp_world_tilted_up"/>
+    </joint>
+    <joint name="gripper_tcp_world_tilted_down_mount" type="fixed">
+        <!-- tilt gripper tcp in world frame by 135 deg to compensate for natural tilt with z-axis looking down -->
+        <origin rpy="0.0 2.35619 0.0" xyz="0.0 0.0 0.0"/>
+        <parent link="gripper_tcp_world"/>
+        <child link="gripper_tcp_world_tilted_down"/>
     </joint>
     <joint name="finger1_joint" type="prismatic">
@@ -526,9 +562,27 @@
         <limit effort="30.0" lower="-0.01" upper="0.036" velocity="0.1"/>
     </joint>
-    <joint name="vacuum_up_to_tcp" type="fixed">
+    <joint name="vacuum_up_tcp_mount" type="fixed">
         <!-- place TCP at the end of the tool (z-direction) -->
         <origin rpy="0.0 0.0 0.0" xyz="0.0 0.0 0.07"/>
         <parent link="vacuum_gripper_up"/>
         <child link="vacuum_up_tcp"/>
+    </joint>
+    <joint name="vacuum_up_tcp_world_mount" type="fixed">
+        <!-- reverse all previous rotations -->
+        <origin rpy="-3.14 -0.785 1.57" xyz="0.0 0.0 0.0"/>
+        <parent link="vacuum_up_tcp"/>
+        <child link="vacuum_up_tcp_world"/>
+    </joint>
+    <joint name="vacuum_up_tcp_world_tilted_up_mount" type="fixed">
+        <!-- tilt gripper tcp in world frame by -45 deg to compensate for natural tilt -->
+        <origin rpy="0.0 -0.785 0.0" xyz="0.0 0.0 0.0"/>
+        <parent link="vacuum_up_tcp_world"/>
+        <child link="vacuum_up_tcp_world_tilted_up"/>
+    </joint>
+    <joint name="vacuum_up_tcp_world_tilted_down_mount" type="fixed">
+        <!-- tilt gripper tcp in world frame by 135 deg to compensate for natural tilt with z-axis looking down -->
+        <origin rpy="0.0 2.35619 0.0" xyz="0.0 0.0 0.0"/>
+        <parent link="vacuum_up_tcp_world"/>
+        <child link="vacuum_up_tcp_world_tilted_down"/>
     </joint>
     <joint name="vacuum_down_joint" type="prismatic">
@@ -539,5 +593,5 @@
         <limit effort="30.0" lower="-0.01" upper="0.036" velocity="0.1"/>
     </joint>
-    <joint name="vacuum_down_to_tcp" type="fixed">
+    <joint name="vacuum_down_tcp_mount" type="fixed">
         <!-- place TCP at the end of the tool (z-direction) -->
         <origin rpy="0.0 0.0 0.0" xyz="0.0 0.0 0.07"/>
@@ -545,3 +599,21 @@
         <child link="vacuum_down_tcp"/>
     </joint>
+    <joint name="vacuum_down_tcp_world_mount" type="fixed">
+        <!-- reverse all previous rotations -->
+        <origin rpy="-3.14 -0.785 1.57" xyz="0.0 0.0 0.0"/>
+        <parent link="vacuum_down_tcp"/>
+        <child link="vacuum_down_tcp_world"/>
+    </joint>
+    <joint name="vacuum_down_tcp_world_tilted_up_mount" type="fixed">
+        <!-- tilt gripper tcp in world frame by -45 deg to compensate for natural tilt -->
+        <origin rpy="0.0 -0.785 0.0" xyz="0.0 0.0 0.0"/>
+        <parent link="vacuum_down_tcp_world"/>
+        <child link="vacuum_down_tcp_world_tilted_up"/>
+    </joint>
+    <joint name="vacuum_down_tcp_world_tilted_down_mount" type="fixed">
+        <!-- tilt gripper tcp in world frame by 135 deg to compensate for natural tilt with z-axis looking down -->
+        <origin rpy="0.0 2.35619 0.0" xyz="0.0 0.0 0.0"/>
+        <parent link="vacuum_down_tcp_world"/>
+        <child link="vacuum_down_tcp_world_tilted_down"/>
+    </joint>
 </robot>

Commit message: increase resolution in rotations

File: src/cobot_model/urdf/robot_model.urdf.xacro (robot description, xacro)
@@ -150,5 +150,5 @@
             </xacro:if>
             <xacro:unless value="${'$(arg use_collision_meshes)' == 'true'}">
-                <origin rpy="1.57 0.0 0.0" xyz="0.0 0.126 0.06"/>
+                <origin rpy="1.5708 0.0 0.0" xyz="0.0 0.126 0.06"/>
                 <geometry>
                     <cylinder radius="0.06" length="0.372"/>
@@ -240,5 +240,5 @@
              </xacro:if>
             <xacro:unless value="${'$(arg use_collision_meshes)' == 'true'}">
-                <origin rpy="0.0 1.57 0.0" xyz="-0.12 0.0 -0.04"/>
+                <origin rpy="0.0 1.5708 0.0" xyz="-0.12 0.0 -0.04"/>
                 <geometry>
                     <cylinder length="0.15" radius="0.04"/>
@@ -270,5 +270,5 @@
             </xacro:if>
             <xacro:unless value="${'$(arg use_collision_meshes)' == 'true'}">
-                <origin rpy="-0.786 0.0 0.0" xyz="0.0 0.1 0.05"/>
+                <origin rpy="-0.785398 0.0 0.0" xyz="0.0 0.1 0.05"/>
                 <geometry>
                     <box size="0.124 0.135 0.14"/>
@@ -280,5 +280,5 @@
             <!-- tilt the inertia tensor by 45 deg to match the actual mesh
                  => same tilt is applied in the tool_base link -->
-            <origin rpy="0.785 0.0 0.0" xyz="0.0 0.09 0.04"/>
+            <origin rpy="0.785398 0.0 0.0" xyz="0.0 0.09 0.04"/>
            <inertia ixx="0.01533367" iyy="0.02185067" izz="0.02693367" ixy="0.0" ixz="0.0" iyz="0.0" />
         </inertial>
@@ -302,5 +302,6 @@
             </xacro:if>
             <xacro:unless value="${'$(arg use_collision_meshes)' == 'true'}">
-                <origin rpy="0.0 -0.25 0.0" xyz="0.046 0.0 0.056"/>
+                <!-- tilt geometric object by 15 deg to match real gripper -->
+                <origin rpy="0.0 -0.261799 0.0" xyz="0.046 0.0 0.056"/>
                 <geometry>
                     <cylinder length="0.10" radius="0.01"/>
@@ -310,7 +311,5 @@
         <inertial>
             <mass value="0.05" />
-            <!-- <origin rpy="-0.785 0.0 0.0" xyz="0.02 0.03 0.03" / -->
-            <origin rpy="0.0 -0.25 0.0" xyz="0.046 0.0 0.056"/>
-            <!-- <origin rpy="0.0 0.0 0.0" xyz="0.0 0.0 0.0" /> -->
+            <origin rpy="0.0 -0.261799 0.0" xyz="0.046 0.0 0.056"/>
             <inertia ixx="3.46666667e-05" iyy="2.64166667e-05" izz="1.78833333e-05" ixy="0.0" ixz="0.0" iyz="0.0" />
         </inertial>
@@ -334,5 +333,5 @@
             </xacro:if>
             <xacro:unless value="${'$(arg use_collision_meshes)' == 'true'}">
-                <origin rpy="0.0 0.25 0.0" xyz="-0.046 0.0 0.056"/>
+                <origin rpy="0.0 0.261799 0.0" xyz="-0.046 0.0 0.056"/>
                 <geometry>
                     <cylinder length="0.10" radius="0.01"/>
@@ -342,5 +341,5 @@
         <inertial>
             <mass value="0.05" />
-            <origin rpy="0.0 0.25 0.0" xyz="-0.046 0.0 0.056"/>
+            <origin rpy="0.0 0.261799 0.0" xyz="-0.046 0.0 0.056"/>
             <inertia ixx="3.46666667e-05" iyy="2.64166667e-05" izz="1.78833333e-05" ixy="0.0" ixz="0.0" iyz="0.0" />
         </inertial>
@@ -445,5 +444,5 @@
         <child link="lin_axis_carriage" />
         <axis xyz="0 0 1" />
-        <limit effort="300.0" velocity="3.141593" lower="-0.001" upper="0.894" />
+        <limit effort="300.0" velocity="3.14159" lower="-0.001" upper="0.894" />
     </joint>
     <joint name="mount_fixture" type="fixed">
@@ -457,13 +456,13 @@
         <child link="segment2" />
         <axis xyz="0 0 1" />
-        <limit effort="200.0" velocity="3.141593" lower="-2.37365" upper="2.37365" />
+        <limit effort="200.0" velocity="3.14159" lower="-2.37365" upper="2.37365" />
         <dynamics damping="0.0" friction="0.0" />
     </joint>
     <joint name="joint_2" type="revolute">
-        <origin rpy="1.57 0.0 0.0" xyz="0.0 -0.111 0.118"/>
+        <origin rpy="1.5708 0.0 0.0" xyz="0.0 -0.111 0.118"/>
         <parent link="segment2" />
         <child link="segment3" />
         <axis xyz="0 0 1" />
-        <limit effort="150.0" velocity="3.141593" lower="-2.26893" upper="0.785398" />
+        <limit effort="150.0" velocity="3.14159" lower="-2.26893" upper="0.785398" />
         <dynamics damping="0.0" friction="0.0" />
     </joint>
@@ -473,29 +472,29 @@
         <child link="segment4" />
         <axis xyz="0 0 1" />
-        <limit effort="100.0" velocity="3.141593" lower="-0.785398" upper="2.26893" />
+        <limit effort="100.0" velocity="3.14159" lower="-0.785398" upper="2.26893" />
         <dynamics damping="0.0" friction="0.0" />
     </joint>
     <joint name="joint_4" type="revolute">
-        <origin rpy="0.0 1.570 0.0" xyz="0.062 0.0 -0.168"/>
+        <origin rpy="0.0 1.5708 0.0" xyz="0.062 0.0 -0.168"/>
         <parent link="segment4" />
         <child link="segment5" />
         <axis xyz="0 0 1" />
-        <limit effort="50.0" velocity="3.141593" lower="-1.570796" upper="1.570796" />
+        <limit effort="50.0" velocity="3.14159" lower="-1.5708" upper="1.5708" />
         <dynamics damping="0.0" friction="0.0" />
     </joint>
     <joint name="joint_5" type="revolute">
-        <origin rpy="0.0 1.57 0.0" xyz="0.042 0.0 0.183"/>
+        <origin rpy="0.0 1.5708 0.0" xyz="0.042 0.0 0.183"/>
         <parent link="segment5" />
         <child link="segment6" />
         <axis xyz="0 0 1" />
-        <limit effort="50.0" velocity="3.141593" lower="-1.570796" upper="1.570796" />
+        <limit effort="50.0" velocity="3.14159" lower="-1.5708" upper="1.5708" />
         <dynamics damping="0.0" friction="0.0" />
     </joint>
     <joint name="joint_6" type="revolute">
-        <origin rpy="0.0 -1.570 0.0" xyz="-0.156 0.0 -0.04"/>
+        <origin rpy="0.0 -1.5708 0.0" xyz="-0.156 0.0 -0.04"/>
         <parent link="segment6"/>
         <child link="segment7"/>
         <axis xyz="0 0 1"/>
-        <limit effort="20." lower="-2.37365" upper="2.37365" velocity="3.141593"/>
+        <limit effort="20." lower="-2.37365" upper="2.37365" velocity="3.14159"/>
         <dynamics damping="0.0" friction="0.0"/>
     </joint>
@@ -512,5 +511,5 @@
     <joint name="tool_mount" type="fixed">
         <!-- tilt tool base by 45 deg + move coordinate frame -->
-        <origin rpy="0.785 0.0 0.0" xyz="0.0 0.072 0.060"/>
+        <origin rpy="0.785398 0.0 0.0" xyz="0.0 0.072 0.060"/>
         <parent link="flange"/>
         <child link="tool_base"/>
@@ -524,5 +523,5 @@
     <joint name="gripper_tcp_world_mount" type="fixed">
         <!-- reverse all previous rotations -->
-        <origin rpy="-3.14 -0.785 1.57" xyz="0.0 0.0 0.0"/>
+        <origin rpy="-3.14159 -0.785398 1.5708" xyz="0.0 0.0 0.0"/>
         <parent link="gripper_tcp"/>
         <child link="gripper_tcp_world"/>
@@ -530,5 +529,5 @@
     <joint name="gripper_tcp_world_tilted_up_mount" type="fixed">
         <!-- tilt gripper tcp in world frame by -45 deg to compensate for natural tilt -->
-        <origin rpy="0.0 -0.785 0.0" xyz="0.0 0.0 0.0"/>
+        <origin rpy="0.0 -0.785398 0.0" xyz="0.0 0.0 0.0"/>
         <parent link="gripper_tcp_world"/>
         <child link="gripper_tcp_world_tilted_up"/>
@@ -570,5 +569,5 @@
     <joint name="vacuum_up_tcp_world_mount" type="fixed">
         <!-- reverse all previous rotations -->
-        <origin rpy="-3.14 -0.785 1.57" xyz="0.0 0.0 0.0"/>
+        <origin rpy="-3.14159 -0.785398 1.5708" xyz="0.0 0.0 0.0"/>
         <parent link="vacuum_up_tcp"/>
         <child link="vacuum_up_tcp_world"/>
@@ -576,5 +575,5 @@
     <joint name="vacuum_up_tcp_world_tilted_up_mount" type="fixed">
         <!-- tilt gripper tcp in world frame by -45 deg to compensate for natural tilt -->
-        <origin rpy="0.0 -0.785 0.0" xyz="0.0 0.0 0.0"/>
+        <origin rpy="0.0 -0.785398 0.0" xyz="0.0 0.0 0.0"/>
         <parent link="vacuum_up_tcp_world"/>
         <child link="vacuum_up_tcp_world_tilted_up"/>
@@ -601,5 +600,5 @@
     <joint name="vacuum_down_tcp_world_mount" type="fixed">
         <!-- reverse all previous rotations -->
-        <origin rpy="-3.14 -0.785 1.57" xyz="0.0 0.0 0.0"/>
+        <origin rpy="-3.14159 -0.785398 1.5708" xyz="0.0 0.0 0.0"/>
         <parent link="vacuum_down_tcp"/>
         <child link="vacuum_down_tcp_world"/>
@@ -607,5 +606,5 @@
     <joint name="vacuum_down_tcp_world_tilted_up_mount" type="fixed">
         <!-- tilt gripper tcp in world frame by -45 deg to compensate for natural tilt -->
-        <origin rpy="0.0 -0.785 0.0" xyz="0.0 0.0 0.0"/>
+        <origin rpy="0.0 -0.785398 0.0" xyz="0.0 0.0 0.0"/>
         <parent link="vacuum_down_tcp_world"/>
         <child link="vacuum_down_tcp_world_tilted_up"/>

Commit message: update vacuum gripper extension value

File: src/cobot_model/urdf/robot_model.urdf.xacro (robot description, xacro)
@@ -559,5 +559,5 @@
         <child link="vacuum_gripper_up"/>
         <axis xyz="0 0 1"/>
-        <limit effort="30.0" lower="-0.01" upper="0.036" velocity="0.1"/>
+        <limit effort="30.0" lower="-0.01" upper="0.055" velocity="0.1"/>
     </joint>
     <joint name="vacuum_up_tcp_mount" type="fixed">
@@ -590,5 +590,5 @@
         <child link="vacuum_gripper_down"/>
         <axis xyz="0 0 1"/>
-        <limit effort="30.0" lower="-0.01" upper="0.036" velocity="0.1"/>
+        <limit effort="30.0" lower="-0.01" upper="0.055" velocity="0.1"/>
     </joint>
     <joint name="vacuum_down_tcp_mount" type="fixed">

Commit message: reference new mesh in urdf

File: src/cobot_model/urdf/robot_model.urdf.xacro (robot description, xacro)
@@ -15,5 +15,5 @@
             <origin rpy="0.0 0.0 0.0" xyz="0.0 0.0 0.0" />
             <geometry>
-                <mesh filename="package://cobot_model/meshes/visual/axis_visual.stl"/>
+                <mesh filename="package://cobot_model/meshes/visual/axis_and_workbench_visual.dae"/>
             </geometry>
             <material name="axis_material">
@@ -25,5 +25,5 @@
                 <origin rpy="0.0 0.0 0.0" xyz="0.0 0.0 0.0" />
                 <geometry>
-                   <mesh filename="package://cobot_model/meshes/collision/axis_collision.stl"/>
+                   <mesh filename="package://cobot_model/meshes/collision/axis_and_workbench_collision.stl"/>
                 </geometry>
             </xacro:if>

Commit message: move cobot by 32cm in z and reference new meshes

File: src/cobot_model/urdf/robot_model.urdf.xacro (robot description, xacro)
@@ -4,5 +4,5 @@
     <link name="world" />
     <joint name="robot_in_world" type="fixed">
-        <origin xyz="0.0 0.0 0.0" rpy="0.0 0.0 0.0" />
+        <origin xyz="0.0 0.0 0.32" rpy="0.0 0.0 0.0" />
         <parent link="world" />
         <child link="base_link" />
@@ -15,5 +15,5 @@
             <origin rpy="0.0 0.0 0.0" xyz="0.0 0.0 0.0" />
             <geometry>
-                <mesh filename="package://cobot_model/meshes/visual/axis_and_workbench_visual.dae"/>
+                <mesh filename="package://cobot_model/meshes/visual/axis_table_workbench_visual.dae"/>
             </geometry>
             <material name="axis_material">
@@ -25,5 +25,5 @@
                 <origin rpy="0.0 0.0 0.0" xyz="0.0 0.0 0.0" />
                 <geometry>
-                   <mesh filename="package://cobot_model/meshes/collision/axis_and_workbench_collision.stl"/>
+                   <mesh filename="package://cobot_model/meshes/collision/axis_table_workbench_collision.stl"/>
                 </geometry>
             </xacro:if>
