Commit message: reference new meshes in xacro

File: src/cobot_model/urdf/robot_model.urdf.xacro (robot description, xacro)
@@ -15,5 +15,5 @@
             <origin rpy="0.0 0.0 0.0" xyz="0.0 0.0 0.0" />
             <geometry>
-                <mesh filename="package://cobot_model/meshes/visual/axis_table_workbench_visual.dae"/>
+                <mesh filename="package://cobot_model/meshes/visual/cobot_base_frame_visual_logo.dae"/>
             </geometry>
             <material name="axis_material">
@@ -25,5 +25,5 @@
                 <origin rpy="0.0 0.0 0.0" xyz="0.0 0.0 0.0" />
                 <geometry>
-                   <mesh filename="package://cobot_model/meshes/collision/axis_table_workbench_collision.stl"/>
+                   <mesh filename="package://cobot_model/meshes/collision/cobot_base_frame_collision.stl"/>
                 </geometry>
             </xacro:if>
